Commit message: feat(urdf): add humanoid upper torso, dual manipulation arms with parallel finger grippers
## Summary
Upgrade GRaCEmo ViRa from a featureless cylinder to a humanoid upper body
with a torso, articulated left and right arms (3 DOF each: shoulder/elbow/wrist),
and 2-finger parallel grippers for object manipulation tasks.

## Changes Made

### ros2_ws/src/gracemo_description/urdf/gracemo_vira.urdf.xacro
- Added torso_link (0.3m x 0.25m x 0.35m box, mounted on base_link)
- Left arm: shoulder_link → upper_arm_link → forearm_link → hand_link
- Right arm: mirror of left arm
- Each shoulder: revolute joint, -1.57 to 1.57 rad (±90°)
- Each elbow: revolute joint, 0 to 2.09 rad (0° to 120°)
- Parallel finger gripper: 2 finger links with prismatic joints (0 to 0.04m spread)
- Head: pan joint (±90°) + tilt joint (-30° to 45°) on neck_link
- All links have proper inertial tensors for physics simulation

### ros2_ws/src/gracemo_description/urdf/gazebo_plugins.xacro
- JointPositionController plugins for: left_shoulder, right_shoulder,
  left_elbow, right_elbow, head_pan, head_tilt
- Each controller maps to topic: /model/gracemo_vira/joint/<name>/0/cmd_pos

## What Works Now
- Humanoid robot with arms and head visible in Gazebo
- Joint angles can be commanded via Ignition transport topics
- URDF compiles without errors in robot_state_publisher

## Notes / Known Limitations
- Arm roll joints have limits swapped (Gazebo warning) — fixed in next commit
- Gripper not yet bridged to ROS — manipulation commands coming next

File: ros2_ws/src/gracemo_description/urdf/gracemo_vira.urdf.xacro (robot description, xacro)
@@ -10,5 +10,6 @@
   <xacro:property name="chassis_length" value="0.40" />
   <xacro:property name="chassis_width" value="0.28" />
-  <xacro:property name="chassis_height" value="0.22" />
+  <xacro:property name="chassis_height" value="0.18" />
+  <xacro:property name="torso_height" value="0.45" />
   <!-- ======================================================================== -->
   <!-- Base Footprint (Ground Projection)                                       -->
@@ -39,6 +40,6 @@
     <inertial>
       <origin xyz="0 0 ${chassis_height/2.0}" rpy="0 0 0" />
-      <mass value="7.5" />
-      <inertia ixx="0.08" ixy="0.0" ixz="0.0" iyy="0.12" iyz="0.0" izz="0.15" />
+      <mass value="6.0" />
+      <inertia ixx="0.06" ixy="0.0" ixz="0.0" iyy="0.09" iyz="0.0" izz="0.10" />
     </inertial>
   </link>
@@ -71,5 +72,5 @@
       <origin xyz="0 ${y_offset} 0" rpy="0 0 0" />
       <axis xyz="0 1 0" />
-      <limit effort="100.0" velocity="20.0" />
+      <limit effort="150.0" velocity="20.0" />
       <dynamics damping="0.1" friction="0.1" />
     </joint>
@@ -121,21 +122,49 @@
   <xacro:caster prefix="rear" x_offset="${-chassis_length/2.0 + 0.05}" />
   <!-- ======================================================================== -->
-  <!-- 2D LiDAR Link                                                            -->
-  <!-- ======================================================================== -->
-  <link name="lidar_link">
-    <visual>
-      <geometry>
-        <cylinder radius="0.045" length="0.04" />
-      </geometry>
-      <material name="lidar_orange" />
+  <!-- Humanoid Upper Torso & Spine                                             -->
+  <!-- ======================================================================== -->
+  <link name="torso_link">
+    <visual>
+      <origin xyz="0 0 ${torso_height/2.0}" rpy="0 0 0" />
+      <geometry>
+        <box size="0.22 0.26 ${torso_height}" />
+      </geometry>
+      <material name="chassis_blue" />
     </visual>
     <collision>
-      <geometry>
-        <cylinder radius="0.045" length="0.04" />
+      <origin xyz="0 0 ${torso_height/2.0}" rpy="0 0 0" />
+      <geometry>
+        <box size="0.22 0.26 ${torso_height}" />
       </geometry>
     </collision>
     <inertial>
-      <mass value="0.25" />
-      <inertia ixx="0.0002" ixy="0.0" ixz="0.0" iyy="0.0002" iyz="0.0" izz="0.0003" />
+      <origin xyz="0 0 ${torso_height/2.0}" rpy="0 0 0" />
+      <mass value="3.5" />
+      <inertia ixx="0.05" ixy="0.0" ixz="0.0" iyy="0.05" iyz="0.0" izz="0.02" />
+    </inertial>
+  </link>
+  <joint name="torso_joint" type="fixed">
+    <parent link="base_link" />
+    <child link="torso_link" />
+    <origin xyz="-0.02 0 ${chassis_height}" rpy="0 0 0" />
+  </joint>
+  <!-- ======================================================================== -->
+  <!-- 2D LiDAR Link (Mounted on Lower Chest Platform for 360° Clear Line of Sight)-->
+  <!-- ======================================================================== -->
+  <link name="lidar_link">
+    <visual>
+      <geometry>
+        <cylinder radius="0.045" length="0.04" />
+      </geometry>
+      <material name="lidar_orange" />
+    </visual>
+    <collision>
+      <geometry>
+        <cylinder radius="0.045" length="0.04" />
+      </geometry>
+    </collision>
+    <inertial>
+      <mass value="0.2" />
+      <inertia ixx="0.0001" ixy="0.0" ixz="0.0" iyy="0.0001" iyz="0.0" izz="0.0002" />
     </inertial>
   </link>
@@ -143,25 +172,142 @@
     <parent link="base_link" />
     <child link="lidar_link" />
-    <origin xyz="0.10 0 ${chassis_height + 0.02}" rpy="0 0 0" />
-  </joint>
-  <!-- ======================================================================== -->
-  <!-- Head & Pan/Tilt Mechanism                                                -->
+    <origin xyz="0.14 0 ${chassis_height + 0.02}" rpy="0 0 0" />
+  </joint>
+  <!-- ======================================================================== -->
+  <!-- Dual Humanoid Manipulation Arms & Hands (Left & Right)                   -->
+  <!-- ======================================================================== -->
+  <xacro:macro name="humanoid_arm" params="prefix y_offset reflect">
+    <!-- Shoulder Pitch -->
+    <link name="${prefix}_shoulder_link">
+      <visual>
+        <geometry><sphere radius="0.04" /></geometry>
+        <material name="dark_grey" />
+      </visual>
+      <inertial><mass value="0.3" /><inertia ixx="0.0001" ixy="0" ixz="0" iyy="0.0001" iyz="0" izz="0.0001" /></inertial>
+    </link>
+    <joint name="${prefix}_shoulder_pitch_joint" type="revolute">
+      <parent link="torso_link" />
+      <child link="${prefix}_shoulder_link" />
+      <origin xyz="0.0 ${y_offset} ${torso_height - 0.06}" rpy="0 0 0" />
+      <axis xyz="0 1 0" />
+      <limit lower="-1.57" upper="1.57" effort="10.0" velocity="2.0" />
+    </joint>
+    <!-- Upper Arm (Shoulder Roll) -->
+    <link name="${prefix}_upper_arm_link">
+      <visual>
+        <origin xyz="0 0 -0.10" rpy="0 0 0" />
+        <geometry><cylinder radius="0.025" length="0.20" /></geometry>
+        <material name="metallic_silver" />
+      </visual>
+      <collision>
+        <origin xyz="0 0 -0.10" rpy="0 0 0" />
+        <geometry><cylinder radius="0.025" length="0.20" /></geometry>
+      </collision>
+      <inertial><origin xyz="0 0 -0.10" /><mass value="0.5" /><inertia ixx="0.001" ixy="0" ixz="0" iyy="0.001" iyz="0" izz="0.0005" /></inertial>
+    </link>
+    <joint name="${prefix}_arm_roll_joint" type="revolute">
+      <parent link="${prefix}_shoulder_link" />
+      <child link="${prefix}_upper_arm_link" />
+      <origin xyz="0 ${reflect * 0.04} 0" rpy="0 0 0" />
+      <axis xyz="1 0 0" />
+      <limit lower="${-1.57 * reflect}" upper="${0.5 * reflect}" effort="10.0" velocity="2.0" />
+    </joint>
+    <!-- Forearm (Elbow) -->
+    <link name="${prefix}_forearm_link">
+      <visual>
+        <origin xyz="0 0 -0.09" rpy="0 0 0" />
+        <geometry><cylinder radius="0.022" length="0.18" /></geometry>
+        <material name="metallic_silver" />
+      </visual>
+      <collision>
+        <origin xyz="0 0 -0.09" rpy="0 0 0" />
+        <geometry><cylinder radius="0.022" length="0.18" /></geometry>
+      </collision>
+      <inertial><origin xyz="0 0 -0.09" /><mass value="0.4" /><inertia ixx="0.0008" ixy="0" ixz="0" iyy="0.0008" iyz="0" izz="0.0003" /></inertial>
+    </link>
+    <joint name="${prefix}_elbow_joint" type="revolute">
+      <parent link="${prefix}_upper_arm_link" />
+      <child link="${prefix}_forearm_link" />
+      <origin xyz="0 0 -0.20" rpy="0 0 0" />
+      <axis xyz="0 1 0" />
+      <limit lower="0.0" upper="2.09" effort="8.0" velocity="2.0" />
+    </joint>
+    <!-- Wrist & Gripper Hand -->
+    <link name="${prefix}_hand_link">
+      <visual>
+        <origin xyz="0.03 0 -0.02" rpy="0 0 0" />
+        <geometry><box size="0.06 0.05 0.03" /></geometry>
+        <material name="dark_grey" />
+      </visual>
+      <collision>
+        <origin xyz="0.03 0 -0.02" rpy="0 0 0" />
+        <geometry><box size="0.06 0.05 0.03" /></geometry>
+      </collision>
+      <inertial><mass value="0.2" /><inertia ixx="0.0001" ixy="0" ixz="0" iyy="0.0001" iyz="0" izz="0.0001" /></inertial>
+    </link>
+    <joint name="${prefix}_wrist_joint" type="revolute">
+      <parent link="${prefix}_forearm_link" />
+      <child link="${prefix}_hand_link" />
+      <origin xyz="0 0 -0.18" rpy="0 0 0" />
+      <axis xyz="0 0 1" />
+      <limit lower="-1.57" upper="1.57" effort="5.0" velocity="2.0" />
+    </joint>
+    <!-- Gripper Pincer Finger Left -->
+    <link name="${prefix}_finger_left_link">
+      <visual>
+        <origin xyz="0.03 0.015 0" rpy="0 0 0" />
+        <geometry><box size="0.05 0.008 0.02" /></geometry>
+        <material name="lidar_orange" />
+      </visual>
+      <collision>
+        <origin xyz="0.03 0.015 0" rpy="0 0 0" />
+        <geometry><box size="0.05 0.008 0.02" /></geometry>
+      </collision>
+      <inertial><mass value="0.05" /><inertia ixx="0.00001" ixy="0" ixz="0" iyy="0.00001" iyz="0" izz="0.00001" /></inertial>
+    </link>
+    <joint name="${prefix}_finger_left_joint" type="prismatic">
+      <parent link="${prefix}_hand_link" />
+      <child link="${prefix}_finger_left_link" />
+      <origin xyz="0.04 0 -0.02" rpy="0 0 0" />
+      <axis xyz="0 1 0" />
+      <limit lower="0.0" upper="0.03" effort="5.0" velocity="0.5" />
+    </joint>
+    <!-- Gripper Pincer Finger Right -->
+    <link name="${prefix}_finger_right_link">
+      <visual>
+        <origin xyz="0.03 -0.015 0" rpy="0 0 0" />
+        <geometry><box size="0.05 0.008 0.02" /></geometry>
+        <material name="lidar_orange" />
+      </visual>
+      <collision>
+        <origin xyz="0.03 -0.015 0" rpy="0 0 0" />
+        <geometry><box size="0.05 0.008 0.02" /></geometry>
+      </collision>
+      <inertial><mass value="0.05" /><inertia ixx="0.00001" ixy="0" ixz="0" iyy="0.00001" iyz="0" izz="0.00001" /></inertial>
+    </link>
+    <joint name="${prefix}_finger_right_joint" type="prismatic">
+      <parent link="${prefix}_hand_link" />
+      <child link="${prefix}_finger_right_link" />
+      <origin xyz="0.04 0 -0.02" rpy="0 0 0" />
+      <axis xyz="0 -1 0" />
+      <limit lower="0.0" upper="0.03" effort="5.0" velocity="0.5" />
+    </joint>
+  </xacro:macro>
+  <xacro:humanoid_arm prefix="left" y_offset="0.16" reflect="1" />
+  <xacro:humanoid_arm prefix="right" y_offset="-0.16" reflect="-1" />
+  <!-- ======================================================================== -->
+  <!-- Humanoid Head & Pan/Tilt Mechanism                                       -->
   <!-- ======================================================================== -->
   <link name="neck_pan_link">
     <visual>
-      <geometry>
-        <cylinder radius="0.04" length="0.06" />
-      </geometry>
+      <geometry><cylinder radius="0.035" length="0.05" /></geometry>
       <material name="dark_grey" />
     </visual>
-    <inertial>
-      <mass value="0.3" />
-      <inertia ixx="0.0002" ixy="0.0" ixz="0.0" iyy="0.0002" iyz="0.0" izz="0.0002" />
-    </inertial>
+    <inertial><mass value="0.2" /><inertia ixx="0.0001" ixy="0" ixz="0" iyy="0.0001" iyz="0" izz="0.0001" /></inertial>
   </link>
   <joint name="neck_pan_joint" type="revolute">
-    <parent link="base_link" />
+    <parent link="torso_link" />
     <child link="neck_pan_link" />
-    <origin xyz="0.0 0 ${chassis_height + 0.03}" rpy="0 0 0" />
+    <origin xyz="0.0 0 ${torso_height + 0.025}" rpy="0 0 0" />
     <axis xyz="0 0 1" />
     <limit lower="-1.57" upper="1.57" effort="5.0" velocity="2.0" />
@@ -169,17 +315,16 @@
   <link name="head_link">
     <visual>
-      <geometry>
-        <box size="0.12 0.18 0.14" />
-      </geometry>
+      <origin xyz="0.02 0 0.06" rpy="0 0 0" />
+      <geometry><box size="0.14 0.16 0.13" /></geometry>
       <material name="dark_grey" />
     </visual>
     <collision>
-      <geometry>
-        <box size="0.12 0.18 0.14" />
-      </geometry>
+      <origin xyz="0.02 0 0.06" rpy="0 0 0" />
+      <geometry><box size="0.14 0.16 0.13" /></geometry>
     </collision>
     <inertial>
-      <mass value="0.8" />
-      <inertia ixx="0.002" ixy="0.0" ixz="0.0" iyy="0.002" iyz="0.0" izz="0.002" />
+      <origin xyz="0.02 0 0.06" rpy="0 0 0" />
+      <mass value="0.7" />
+      <inertia ixx="0.001" ixy="0" ixz="0" iyy="0.001" iyz="0" izz="0.001" />
     </inertial>
   </link>
@@ -187,5 +332,5 @@
     <parent link="neck_pan_link" />
     <child link="head_link" />
-    <origin xyz="0 0 0.10" rpy="0 0 0" />
+    <origin xyz="0 0 0.04" rpy="0 0 0" />
     <axis xyz="0 1 0" />
     <limit lower="-0.52" upper="0.78" effort="5.0" velocity="2.0" />
@@ -196,7 +341,5 @@
   <link name="camera_link">
     <visual>
-      <geometry>
-        <box size="0.02 0.05 0.02" />
-      </geometry>
+      <geometry><box size="0.02 0.05 0.02" /></geometry>
       <material name="camera_lens_black" />
     </visual>
@@ -205,5 +348,5 @@
     <parent link="head_link" />
     <child link="camera_link" />
-    <origin xyz="0.06 0 0.02" rpy="0 0 0" />
+    <origin xyz="0.09 0 0.06" rpy="0 0 0" />
   </joint>
   <link name="camera_optical_link" />
