Commit message: fix(sim): clean visual geometries and synchronize apartment world with unified robot
## Summary
- Re-architected robot links to use single cohesive geometric shapes per link instead of scattered floating sub-primitives.
- Cleaned up embed_robot_world.py to remove old duplicate model comments and ensure world file contains the single unified model definition.
- Positioned default GUI camera at an optimal close-up 3D isometric angle (-2.5, -4.5, 3.5) directly focused on the robot.

## What Works Now
- Complete, unified robot body (chassis, wheels, casters, torso, screen, LiDAR, head, visor, camera, arms) cleanly rendered without floating parts.
- Immediate 3D perspective camera focused on the robot upon Gazebo start.

File: ros2_ws/src/gracemo_description/urdf/gracemo_vira.urdf.xacro (robot description, xacro)
@@ -7,11 +7,11 @@
   <xacro:property name="wheel_radius" value="0.065" />
   <xacro:property name="wheel_width" value="0.035" />
-  <xacro:property name="wheelbase" value="0.32" />
-  <xacro:property name="chassis_length" value="0.38" />
-  <xacro:property name="chassis_width" value="0.26" />
-  <xacro:property name="chassis_height" value="0.12" />
-  <xacro:property name="torso_height" value="0.40" />
-  <xacro:property name="torso_width" value="0.22" />
-  <xacro:property name="torso_depth" value="0.18" />
+  <xacro:property name="wheelbase" value="0.33" />
+  <xacro:property name="chassis_l" value="0.40" />
+  <xacro:property name="chassis_w" value="0.28" />
+  <xacro:property name="chassis_h" value="0.14" />
+  <xacro:property name="torso_l" value="0.20" />
+  <xacro:property name="torso_w" value="0.22" />
+  <xacro:property name="torso_h" value="0.38" />
   <!-- ======================================================================== -->
   <!-- Base Footprint (Ground Projection)                                       -->
@@ -27,30 +27,30 @@
   <!-- ======================================================================== -->
   <link name="base_link">
-    <!-- Main Chassis Body -->
-    <visual>
-      <origin xyz="0 0 ${chassis_height/2.0}" rpy="0 0 0" />
-      <geometry>
-        <box size="${chassis_length} ${chassis_width} ${chassis_height}" />
+    <!-- Main Chassis Box -->
+    <visual>
+      <origin xyz="0 0 ${chassis_h/2.0}" rpy="0 0 0" />
+      <geometry>
+        <box size="${chassis_l} ${chassis_w} ${chassis_h}" />
       </geometry>
       <material name="chassis_blue" />
     </visual>
     <collision>
-      <origin xyz="0 0 ${chassis_height/2.0}" rpy="0 0 0" />
-      <geometry>
-        <box size="${chassis_length} ${chassis_width} ${chassis_height}" />
+      <origin xyz="0 0 ${chassis_h/2.0}" rpy="0 0 0" />
+      <geometry>
+        <box size="${chassis_l} ${chassis_w} ${chassis_h}" />
       </geometry>
     </collision>
-    <!-- Top accent plate -->
-    <visual>
-      <origin xyz="0 0 ${chassis_height + 0.005}" rpy="0 0 0" />
-      <geometry>
-        <box size="${chassis_length - 0.04} ${chassis_width - 0.04} 0.01" />
+    <!-- Bumper Trim Front -->
+    <visual>
+      <origin xyz="${chassis_l/2.0} 0 ${chassis_h/2.0}" rpy="0 0 0" />
+      <geometry>
+        <box size="0.02 ${chassis_w + 0.01} ${chassis_h - 0.02}" />
       </geometry>
       <material name="dark_grey" />
     </visual>
     <inertial>
-      <origin xyz="0 0 ${chassis_height/2.0}" rpy="0 0 0" />
+      <origin xyz="0 0 ${chassis_h/2.0}" rpy="0 0 0" />
       <mass value="6.0" />
-      <inertia ixx="0.06" ixy="0.0" ixz="0.0" iyy="0.08" iyz="0.0" izz="0.10" />
+      <inertia ixx="0.05" ixy="0.0" ixz="0.0" iyy="0.09" iyz="0.0" izz="0.11" />
     </inertial>
   </link>
@@ -66,12 +66,4 @@
         </geometry>
         <material name="rubber_black" />
-      </visual>
-      <!-- Wheel rim accent -->
-      <visual>
-        <origin xyz="0 0 0" rpy="${pi/2} 0 0" />
-        <geometry>
-          <cylinder radius="${wheel_radius * 0.6}" length="${wheel_width + 0.002}" />
-        </geometry>
-        <material name="metallic_silver" />
       </visual>
       <collision>
@@ -97,6 +89,4 @@
       <mu1>1.5</mu1>
       <mu2>1.5</mu2>
-      <kp>1000000.0</kp>
-      <kd>100.0</kd>
       <material>Gazebo/DarkGrey</material>
     </gazebo>
@@ -136,34 +126,34 @@
     </gazebo>
   </xacro:macro>
-  <xacro:caster prefix="front" x_offset="${chassis_length/2.0 - 0.05}" />
-  <xacro:caster prefix="rear" x_offset="${-chassis_length/2.0 + 0.05}" />
-  <!-- ======================================================================== -->
-  <!-- Upper Torso & Humanoid Body                                              -->
+  <xacro:caster prefix="front" x_offset="${chassis_l/2.0 - 0.05}" />
+  <xacro:caster prefix="rear" x_offset="${-chassis_l/2.0 + 0.05}" />
+  <!-- ======================================================================== -->
+  <!-- Torso & Humanoid Body Column                                             -->
   <!-- ======================================================================== -->
   <link name="torso_link">
-    <!-- Main Chest / Torso Body -->
-    <visual>
-      <origin xyz="0 0 ${torso_height/2.0}" rpy="0 0 0" />
-      <geometry>
-        <box size="${torso_depth} ${torso_width} ${torso_height}" />
+    <!-- Torso Column -->
+    <visual>
+      <origin xyz="0 0 ${torso_h/2.0}" rpy="0 0 0" />
+      <geometry>
+        <box size="${torso_l} ${torso_w} ${torso_h}" />
       </geometry>
       <material name="chassis_blue" />
     </visual>
     <collision>
-      <origin xyz="0 0 ${torso_height/2.0}" rpy="0 0 0" />
-      <geometry>
-        <box size="${torso_depth} ${torso_width} ${torso_height}" />
+      <origin xyz="0 0 ${torso_h/2.0}" rpy="0 0 0" />
+      <geometry>
+        <box size="${torso_l} ${torso_w} ${torso_h}" />
       </geometry>
     </collision>
-    <!-- Chest Screen / Accent Panel -->
-    <visual>
-      <origin xyz="${torso_depth/2.0 + 0.005} 0 ${torso_height * 0.6}" rpy="0 0 0" />
-      <geometry>
-        <box size="0.01 0.14 0.12" />
+    <!-- Chest Screen Display -->
+    <visual>
+      <origin xyz="${torso_l/2.0 + 0.005} 0 ${torso_h * 0.6}" rpy="0 0 0" />
+      <geometry>
+        <box size="0.008 0.14 0.12" />
       </geometry>
       <material name="dark_grey" />
     </visual>
     <inertial>
-      <origin xyz="0 0 ${torso_height/2.0}" rpy="0 0 0" />
+      <origin xyz="0 0 ${torso_h/2.0}" rpy="0 0 0" />
       <mass value="3.5" />
       <inertia ixx="0.04" ixy="0.0" ixz="0.0" iyy="0.04" iyz="0.0" izz="0.02" />
@@ -173,23 +163,26 @@
     <parent link="base_link" />
     <child link="torso_link" />
-    <origin xyz="-0.02 0 ${chassis_height}" rpy="0 0 0" />
-  </joint>
-  <!-- ======================================================================== -->
-  <!-- 2D LiDAR (Chest Platform Front)                                          -->
+    <origin xyz="-0.02 0 ${chassis_h}" rpy="0 0 0" />
+  </joint>
+  <!-- ======================================================================== -->
+  <!-- 2D LiDAR (Front Chest Deck)                                              -->
   <!-- ======================================================================== -->
   <link name="lidar_link">
     <visual>
-      <geometry>
-        <cylinder radius="0.04" length="0.035" />
+      <origin xyz="0 0 0.02" rpy="0 0 0" />
+      <geometry>
+        <cylinder radius="0.045" length="0.04" />
       </geometry>
       <material name="lidar_orange" />
     </visual>
     <collision>
-      <geometry>
-        <cylinder radius="0.04" length="0.035" />
+      <origin xyz="0 0 0.02" rpy="0 0 0" />
+      <geometry>
+        <cylinder radius="0.045" length="0.04" />
       </geometry>
     </collision>
     <inertial>
-      <mass value="0.2" />
+      <origin xyz="0 0 0.02" rpy="0 0 0" />
+      <mass value="0.25" />
       <inertia ixx="0.0001" ixy="0.0" ixz="0.0" iyy="0.0001" iyz="0.0" izz="0.0002" />
     </inertial>
@@ -198,15 +191,15 @@
     <parent link="base_link" />
     <child link="lidar_link" />
-    <origin xyz="0.14 0 ${chassis_height + 0.02}" rpy="0 0 0" />
-  </joint>
-  <!-- ======================================================================== -->
-  <!-- Humanoid Head & Visor                                                    -->
+    <origin xyz="${chassis_l/2.0 - 0.06} 0 ${chassis_h}" rpy="0 0 0" />
+  </joint>
+  <!-- ======================================================================== -->
+  <!-- Head & Camera Visor                                                      -->
   <!-- ======================================================================== -->
   <link name="head_link">
-    <!-- Neck -->
+    <!-- Neck Collar -->
     <visual>
       <origin xyz="0 0 0.02" rpy="0 0 0" />
       <geometry>
-        <cylinder radius="0.035" length="0.04" />
+        <cylinder radius="0.04" length="0.04" />
       </geometry>
       <material name="dark_grey" />
@@ -214,26 +207,26 @@
     <!-- Head Unit -->
     <visual>
+      <origin xyz="0.01 0 0.10" rpy="0 0 0" />
+      <geometry>
+        <box size="0.14 0.16 0.12" />
+      </geometry>
+      <material name="chassis_blue" />
+    </visual>
+    <collision>
+      <origin xyz="0.01 0 0.10" rpy="0 0 0" />
+      <geometry>
+        <box size="0.14 0.16 0.12" />
+      </geometry>
+    </collision>
+    <!-- Dark Glass Face Visor -->
+    <visual>
+      <origin xyz="0.082 0 0.10" rpy="0 0 0" />
+      <geometry>
+        <box size="0.006 0.13 0.07" />
+      </geometry>
+      <material name="camera_lens_black" />
+    </visual>
+    <inertial>
       <origin xyz="0.01 0 0.09" rpy="0 0 0" />
-      <geometry>
-        <box size="0.13 0.16 0.11" />
-      </geometry>
-      <material name="chassis_blue" />
-    </visual>
-    <collision>
-      <origin xyz="0.01 0 0.09" rpy="0 0 0" />
-      <geometry>
-        <box size="0.13 0.16 0.11" />
-      </geometry>
-    </collision>
-    <!-- Dark Visor / Face Display -->
-    <visual>
-      <origin xyz="0.076 0 0.09" rpy="0 0 0" />
-      <geometry>
-        <box size="0.006 0.13 0.07" />
-      </geometry>
-      <material name="camera_lens_black" />
-    </visual>
-    <inertial>
-      <origin xyz="0.01 0 0.08" rpy="0 0 0" />
       <mass value="0.8" />
       <inertia ixx="0.001" ixy="0.0" ixz="0.0" iyy="0.001" iyz="0.0" izz="0.001" />
@@ -243,7 +236,7 @@
     <parent link="torso_link" />
     <child link="head_link" />
-    <origin xyz="0 0 ${torso_height}" rpy="0 0 0" />
-  </joint>
-  <!-- Camera Link (Inside Head Visor) -->
+    <origin xyz="0 0 ${torso_h}" rpy="0 0 0" />
+  </joint>
+  <!-- Camera Link (Front Eye) -->
   <link name="camera_link">
     <visual>
@@ -252,5 +245,5 @@
         <cylinder radius="0.012" length="0.01" />
       </geometry>
-      <material name="dark_grey" />
+      <material name="metallic_silver" />
     </visual>
   </link>
@@ -258,5 +251,5 @@
     <parent link="head_link" />
     <child link="camera_link" />
-    <origin xyz="0.08 0 0.09" rpy="0 0 0" />
+    <origin xyz="0.086 0 0.10" rpy="0 0 0" />
   </joint>
   <link name="camera_optical_link" />
@@ -267,57 +260,42 @@
   </joint>
   <!-- ======================================================================== -->
-  <!-- Humanoid Arms (Left & Right - Solid Anatomical Structure)                -->
-  <!-- ======================================================================== -->
-  <xacro:macro name="humanoid_arm" params="prefix y_offset reflect">
+  <!-- Left & Right Humanoid Arms (Clean Integrated Design)                     -->
+  <!-- ======================================================================== -->
+  <xacro:macro name="arm" params="prefix y_offset">
     <link name="${prefix}_arm_link">
-      <!-- Shoulder Joint sphere -->
-      <visual>
-        <origin xyz="0 0 0" rpy="0 0 0" />
-        <geometry><sphere radius="0.035" /></geometry>
+      <!-- Upper Arm -->
+      <visual>
+        <origin xyz="0 0 -0.09" rpy="0 0 0" />
+        <geometry>
+          <box size="0.05 0.04 0.18" />
+        </geometry>
+        <material name="metallic_silver" />
+      </visual>
+      <!-- Forearm & Gripper -->
+      <visual>
+        <origin xyz="0.03 0 -0.22" rpy="0 0.25 0" />
+        <geometry>
+          <box size="0.045 0.035 0.14" />
+        </geometry>
         <material name="dark_grey" />
       </visual>
-      <!-- Upper Arm (pointing down along torso) -->
-      <visual>
-        <origin xyz="0 0 -0.09" rpy="0 0 0" />
-        <geometry><cylinder radius="0.022" length="0.16" /></geometry>
-        <material name="metallic_silver" />
-      </visual>
-      <!-- Elbow Joint sphere -->
-      <visual>
-        <origin xyz="0 0 -0.17" rpy="0 0 0" />
-        <geometry><sphere radius="0.025" /></geometry>
-        <material name="dark_grey" />
-      </visual>
-      <!-- Forearm (angled slightly forward) -->
-      <visual>
-        <origin xyz="0.04 0 -0.23" rpy="0 0.4 0" />
-        <geometry><cylinder radius="0.020" length="0.14" /></geometry>
-        <material name="metallic_silver" />
-      </visual>
-      <!-- Hand / Gripper unit -->
-      <visual>
-        <origin xyz="0.09 0 -0.28" rpy="0 0.4 0" />
-        <geometry><box size="0.04 0.035 0.03" /></geometry>
-        <material name="dark_grey" />
-      </visual>
-      <!-- Pincer fingers -->
-      <visual>
-        <origin xyz="0.115 0.01 -0.29" rpy="0 0.4 0" />
-        <geometry><box size="0.025 0.006 0.012" /></geometry>
+      <!-- Gripper Hand Accent -->
+      <visual>
+        <origin xyz="0.065 0 -0.28" rpy="0 0.25 0" />
+        <geometry>
+          <box size="0.03 0.03 0.02" />
+        </geometry>
         <material name="lidar_orange" />
       </visual>
-      <visual>
-        <origin xyz="0.115 -0.01 -0.29" rpy="0 0.4 0" />
-        <geometry><box size="0.025 0.006 0.012" /></geometry>
-        <material name="lidar_orange" />
-      </visual>
       <collision>
-        <origin xyz="0.03 0 -0.15" rpy="0 0 0" />
-        <geometry><box size="0.08 0.06 0.32" /></geometry>
+        <origin xyz="0.02 0 -0.16" rpy="0 0 0" />
+        <geometry>
+          <box size="0.07 0.05 0.32" />
+        </geometry>
       </collision>
       <inertial>
-        <origin xyz="0.03 0 -0.15" rpy="0 0 0" />
-        <mass value="0.8" />
-        <inertia ixx="0.003" ixy="0.0" ixz="0.0" iyy="0.003" iyz="0.0" izz="0.001" />
+        <origin xyz="0.02 0 -0.16" rpy="0 0 0" />
+        <mass value="0.7" />
+        <inertia ixx="0.002" ixy="0.0" ixz="0.0" iyy="0.002" iyz="0.0" izz="0.001" />
       </inertial>
     </link>
@@ -325,9 +303,9 @@
       <parent link="torso_link" />
       <child link="${prefix}_arm_link" />
-      <origin xyz="0.0 ${y_offset} ${torso_height - 0.04}" rpy="0 0 0" />
+      <origin xyz="0.0 ${y_offset} ${torso_h - 0.04}" rpy="0 0 0" />
     </joint>
   </xacro:macro>
-  <xacro:humanoid_arm prefix="left" y_offset="${torso_width/2.0 + 0.035}" reflect="1" />
-  <xacro:humanoid_arm prefix="right" y_offset="${-torso_width/2.0 - 0.035}" reflect="-1" />
+  <xacro:arm prefix="left" y_offset="${torso_w/2.0 + 0.025}" />
+  <xacro:arm prefix="right" y_offset="${-torso_w/2.0 - 0.025}" />
   <!-- ======================================================================== -->
   <!-- IMU Link                                                                 -->
