Commit message: feat(sim): sleek robot redesign & photorealistic 3D apartment environment in Harmonic
## Summary
1. Redesigned gracemo_vira into a sleek, cohesive, modern humanoid service robot:
   - Replaced scattered primitive boxes with a cylindrical mobile base, dark protective skirt, upright humanoid torso, dark visor face with optical camera eye, seated orange LiDAR dome, and integrated arm pods.
   - Clean rigid anatomy prevents gravity drooping and physics limb explosion.
2. Upgraded apartment environment with photorealistic 3D models:
   - Master Bed (PBR DAE with albedo/normal/roughness textures) in Bedroom.
   - 3D Refrigerator, 3D Dining Table, and 3D Chairs in Kitchen.
   - 3D Sofa, Coffee Table, TV Unit, and 3D Bowl in Living Room.
   - 3D Bookshelf, Desk, Monitor, 3D Cardboard Box, and 3D Coke Can in Study.
   - Clean 4-room layout connected via 2m wide central hallway.
3. Enhanced launch pipeline:
   - Configured GZ_SIM_RESOURCE_PATH for local and fuel models.
   - Positioned default GUI camera at close-up 3D isometric view (-2.5, -4.5, 3.5).

## What Works Now
- High-resolution 3D models render cleanly in Gazebo Harmonic 8 without crashes.
- Unified, sleek humanoid robot sits on the hallway floor at (0, 0, 0.025).
- All ROS 2 topics (/cmd_vel, /odom, /scan, /camera/image_raw, /imu/data, /joint_states, /tf) active.

File: ros2_ws/src/gracemo_description/urdf/gracemo_vira.urdf.xacro (robot description, xacro)
@@ -7,11 +7,10 @@
   <xacro:property name="wheel_radius" value="0.065" />
   <xacro:property name="wheel_width" value="0.035" />
-  <xacro:property name="wheelbase" value="0.33" />
-  <xacro:property name="chassis_l" value="0.40" />
-  <xacro:property name="chassis_w" value="0.28" />
-  <xacro:property name="chassis_h" value="0.14" />
-  <xacro:property name="torso_l" value="0.20" />
-  <xacro:property name="torso_w" value="0.22" />
-  <xacro:property name="torso_h" value="0.38" />
+  <xacro:property name="wheelbase" value="0.32" />
+  <xacro:property name="chassis_radius" value="0.20" />
+  <xacro:property name="chassis_height" value="0.14" />
+  <xacro:property name="torso_height" value="0.40" />
+  <xacro:property name="torso_width" value="0.22" />
+  <xacro:property name="torso_depth" value="0.18" />
   <!-- ======================================================================== -->
   <!-- Base Footprint (Ground Projection)                                       -->
@@ -24,40 +23,49 @@
   </joint>
   <!-- ======================================================================== -->
-  <!-- Base Link (Chassis Body)                                                 -->
+  <!-- Base Link (Sleek Cylindrical Mobile Chassis)                             -->
   <!-- ======================================================================== -->
   <link name="base_link">
-    <!-- Main Chassis Box -->
-    <visual>
-      <origin xyz="0 0 ${chassis_h/2.0}" rpy="0 0 0" />
-      <geometry>
-        <box size="${chassis_l} ${chassis_w} ${chassis_h}" />
+    <!-- Main Cylindrical Chassis Shell -->
+    <visual>
+      <origin xyz="0 0 ${chassis_height/2.0}" rpy="0 0 0" />
+      <geometry>
+        <cylinder radius="${chassis_radius}" length="${chassis_height}" />
       </geometry>
       <material name="chassis_blue" />
     </visual>
+    <!-- Lower Protective Skirt Ring -->
+    <visual>
+      <origin xyz="0 0 ${chassis_height * 0.2}" rpy="0 0 0" />
+      <geometry>
+        <cylinder radius="${chassis_radius + 0.005}" length="${chassis_height * 0.35}" />
+      </geometry>
+      <material name="dark_grey" />
+    </visual>
+    <!-- Top Deck Accent Plate -->
+    <visual>
+      <origin xyz="0 0 ${chassis_height + 0.005}" rpy="0 0 0" />
+      <geometry>
+        <cylinder radius="${chassis_radius * 0.9}" length="0.01" />
+      </geometry>
+      <material name="dark_grey" />
+    </visual>
     <collision>
-      <origin xyz="0 0 ${chassis_h/2.0}" rpy="0 0 0" />
-      <geometry>
-        <box size="${chassis_l} ${chassis_w} ${chassis_h}" />
+      <origin xyz="0 0 ${chassis_height/2.0}" rpy="0 0 0" />
+      <geometry>
+        <cylinder radius="${chassis_radius}" length="${chassis_height}" />
       </geometry>
     </collision>
-    <!-- Bumper Trim Front -->
-    <visual>
-      <origin xyz="${chassis_l/2.0} 0 ${chassis_h/2.0}" rpy="0 0 0" />
-      <geometry>
-        <box size="0.02 ${chassis_w + 0.01} ${chassis_h - 0.02}" />
-      </geometry>
-      <material name="dark_grey" />
-    </visual>
     <inertial>
-      <origin xyz="0 0 ${chassis_h/2.0}" rpy="0 0 0" />
-      <mass value="6.0" />
-      <inertia ixx="0.05" ixy="0.0" ixz="0.0" iyy="0.09" iyz="0.0" izz="0.11" />
+      <origin xyz="0 0 ${chassis_height/2.0}" rpy="0 0 0" />
+      <mass value="6.5" />
+      <inertia ixx="0.07" ixy="0.0" ixz="0.0" iyy="0.07" iyz="0.0" izz="0.12" />
     </inertial>
   </link>
   <!-- ======================================================================== -->
-  <!-- Drive Wheels (Left & Right)                                              -->
+  <!-- Drive Wheels (Left & Right - Recessed in Wheel Wells)                     -->
   <!-- ======================================================================== -->
   <xacro:macro name="wheel" params="prefix y_offset">
     <link name="${prefix}_wheel_link">
+      <!-- Rubber Tire -->
       <visual>
         <origin xyz="0 0 0" rpy="${pi/2} 0 0" />
@@ -66,4 +74,12 @@
         </geometry>
         <material name="rubber_black" />
+      </visual>
+      <!-- Metallic Silver Rim Hub -->
+      <visual>
+        <origin xyz="0 0 0" rpy="${pi/2} 0 0" />
+        <geometry>
+          <cylinder radius="${wheel_radius * 0.6}" length="${wheel_width + 0.002}" />
+        </geometry>
+        <material name="metallic_silver" />
       </visual>
       <collision>
@@ -95,5 +111,5 @@
   <xacro:wheel prefix="right" y_offset="${-wheelbase/2.0}" />
   <!-- ======================================================================== -->
-  <!-- Support Casters (Front & Rear)                                           -->
+  <!-- Support Casters (Front & Rear Spheres)                                   -->
   <!-- ======================================================================== -->
   <xacro:macro name="caster" params="prefix x_offset">
@@ -126,34 +142,34 @@
     </gazebo>
   </xacro:macro>
-  <xacro:caster prefix="front" x_offset="${chassis_l/2.0 - 0.05}" />
-  <xacro:caster prefix="rear" x_offset="${-chassis_l/2.0 + 0.05}" />
-  <!-- ======================================================================== -->
-  <!-- Torso & Humanoid Body Column                                             -->
+  <xacro:caster prefix="front" x_offset="${chassis_radius - 0.06}" />
+  <xacro:caster prefix="rear" x_offset="${-chassis_radius + 0.06}" />
+  <!-- ======================================================================== -->
+  <!-- Humanoid Torso (Center Column & Chest Status Display)                     -->
   <!-- ======================================================================== -->
   <link name="torso_link">
-    <!-- Torso Column -->
-    <visual>
-      <origin xyz="0 0 ${torso_h/2.0}" rpy="0 0 0" />
-      <geometry>
-        <box size="${torso_l} ${torso_w} ${torso_h}" />
+    <!-- Torso Column Body -->
+    <visual>
+      <origin xyz="0 0 ${torso_height/2.0}" rpy="0 0 0" />
+      <geometry>
+        <box size="${torso_depth} ${torso_width} ${torso_height}" />
       </geometry>
       <material name="chassis_blue" />
     </visual>
+    <!-- Chest Glass Status Screen -->
+    <visual>
+      <origin xyz="${torso_depth/2.0 + 0.004} 0 ${torso_height * 0.6}" rpy="0 0 0" />
+      <geometry>
+        <box size="0.006 0.14 0.12" />
+      </geometry>
+      <material name="camera_lens_black" />
+    </visual>
     <collision>
-      <origin xyz="0 0 ${torso_h/2.0}" rpy="0 0 0" />
-      <geometry>
-        <box size="${torso_l} ${torso_w} ${torso_h}" />
+      <origin xyz="0 0 ${torso_height/2.0}" rpy="0 0 0" />
+      <geometry>
+        <box size="${torso_depth} ${torso_width} ${torso_height}" />
       </geometry>
     </collision>
-    <!-- Chest Screen Display -->
-    <visual>
-      <origin xyz="${torso_l/2.0 + 0.005} 0 ${torso_h * 0.6}" rpy="0 0 0" />
-      <geometry>
-        <box size="0.008 0.14 0.12" />
-      </geometry>
-      <material name="dark_grey" />
-    </visual>
     <inertial>
-      <origin xyz="0 0 ${torso_h/2.0}" rpy="0 0 0" />
+      <origin xyz="0 0 ${torso_height/2.0}" rpy="0 0 0" />
       <mass value="3.5" />
       <inertia ixx="0.04" ixy="0.0" ixz="0.0" iyy="0.04" iyz="0.0" izz="0.02" />
@@ -163,14 +179,23 @@
     <parent link="base_link" />
     <child link="torso_link" />
-    <origin xyz="-0.02 0 ${chassis_h}" rpy="0 0 0" />
-  </joint>
-  <!-- ======================================================================== -->
-  <!-- 2D LiDAR (Front Chest Deck)                                              -->
+    <origin xyz="-0.02 0 ${chassis_height}" rpy="0 0 0" />
+  </joint>
+  <!-- ======================================================================== -->
+  <!-- 2D LiDAR (Mounted on Front Deck Platform)                                -->
   <!-- ======================================================================== -->
   <link name="lidar_link">
-    <visual>
-      <origin xyz="0 0 0.02" rpy="0 0 0" />
-      <geometry>
-        <cylinder radius="0.045" length="0.04" />
+    <!-- LiDAR Base Turret -->
+    <visual>
+      <origin xyz="0 0 0.015" rpy="0 0 0" />
+      <geometry>
+        <cylinder radius="0.045" length="0.03" />
+      </geometry>
+      <material name="dark_grey" />
+    </visual>
+    <!-- LiDAR Spinning Ring -->
+    <visual>
+      <origin xyz="0 0 0.032" rpy="0 0 0" />
+      <geometry>
+        <cylinder radius="0.04" length="0.015" />
       </geometry>
       <material name="lidar_orange" />
@@ -191,11 +216,11 @@
     <parent link="base_link" />
     <child link="lidar_link" />
-    <origin xyz="${chassis_l/2.0 - 0.06} 0 ${chassis_h}" rpy="0 0 0" />
-  </joint>
-  <!-- ======================================================================== -->
-  <!-- Head & Camera Visor                                                      -->
+    <origin xyz="0.13 0 ${chassis_height}" rpy="0 0 0" />
+  </joint>
+  <!-- ======================================================================== -->
+  <!-- Humanoid Head & Visor                                                    -->
   <!-- ======================================================================== -->
   <link name="head_link">
-    <!-- Neck Collar -->
+    <!-- Neck Joint -->
     <visual>
       <origin xyz="0 0 0.02" rpy="0 0 0" />
@@ -205,28 +230,28 @@
       <material name="dark_grey" />
     </visual>
-    <!-- Head Unit -->
-    <visual>
-      <origin xyz="0.01 0 0.10" rpy="0 0 0" />
-      <geometry>
-        <box size="0.14 0.16 0.12" />
+    <!-- Rounded Head Shell -->
+    <visual>
+      <origin xyz="0.01 0 0.09" rpy="0 0 0" />
+      <geometry>
+        <box size="0.14 0.16 0.11" />
       </geometry>
       <material name="chassis_blue" />
     </visual>
+    <!-- Dark Glass Face Visor -->
+    <visual>
+      <origin xyz="0.081 0 0.09" rpy="0 0 0" />
+      <geometry>
+        <box size="0.006 0.13 0.07" />
+      </geometry>
+      <material name="camera_lens_black" />
+    </visual>
     <collision>
-      <origin xyz="0.01 0 0.10" rpy="0 0 0" />
-      <geometry>
-        <box size="0.14 0.16 0.12" />
+      <origin xyz="0.01 0 0.09" rpy="0 0 0" />
+      <geometry>
+        <box size="0.14 0.16 0.11" />
       </geometry>
     </collision>
-    <!-- Dark Glass Face Visor -->
-    <visual>
-      <origin xyz="0.082 0 0.10" rpy="0 0 0" />
-      <geometry>
-        <box size="0.006 0.13 0.07" />
-      </geometry>
-      <material name="camera_lens_black" />
-    </visual>
     <inertial>
-      <origin xyz="0.01 0 0.09" rpy="0 0 0" />
+      <origin xyz="0.01 0 0.08" rpy="0 0 0" />
       <mass value="0.8" />
       <inertia ixx="0.001" ixy="0.0" ixz="0.0" iyy="0.001" iyz="0.0" izz="0.001" />
@@ -236,7 +261,7 @@
     <parent link="torso_link" />
     <child link="head_link" />
-    <origin xyz="0 0 ${torso_h}" rpy="0 0 0" />
-  </joint>
-  <!-- Camera Link (Front Eye) -->
+    <origin xyz="0 0 ${torso_height}" rpy="0 0 0" />
+  </joint>
+  <!-- Camera Link (Front Centered Optical Eye) -->
   <link name="camera_link">
     <visual>
@@ -251,5 +276,5 @@
     <parent link="head_link" />
     <child link="camera_link" />
-    <origin xyz="0.086 0 0.10" rpy="0 0 0" />
+    <origin xyz="0.085 0 0.09" rpy="0 0 0" />
   </joint>
   <link name="camera_optical_link" />
@@ -260,21 +285,21 @@
   </joint>
   <!-- ======================================================================== -->
-  <!-- Left & Right Humanoid Arms (Clean Integrated Design)                     -->
+  <!-- Left & Right Manipulation Arm Pods (Sleek Anatomical Integration)        -->
   <!-- ======================================================================== -->
   <xacro:macro name="arm" params="prefix y_offset">
     <link name="${prefix}_arm_link">
-      <!-- Upper Arm -->
+      <!-- Upper Arm Column -->
       <visual>
         <origin xyz="0 0 -0.09" rpy="0 0 0" />
         <geometry>
-          <box size="0.05 0.04 0.18" />
+          <box size="0.045 0.035 0.18" />
         </geometry>
         <material name="metallic_silver" />
       </visual>
-      <!-- Forearm & Gripper -->
-      <visual>
-        <origin xyz="0.03 0 -0.22" rpy="0 0.25 0" />
-        <geometry>
-          <box size="0.045 0.035 0.14" />
+      <!-- Forearm Section -->
+      <visual>
+        <origin xyz="0.025 0 -0.21" rpy="0 0.2 0" />
+        <geometry>
+          <box size="0.04 0.03 0.13" />
         </geometry>
         <material name="dark_grey" />
@@ -282,18 +307,18 @@
       <!-- Gripper Hand Accent -->
       <visual>
-        <origin xyz="0.065 0 -0.28" rpy="0 0.25 0" />
-        <geometry>
-          <box size="0.03 0.03 0.02" />
+        <origin xyz="0.055 0 -0.27" rpy="0 0.2 0" />
+        <geometry>
+          <box size="0.03 0.025 0.02" />
         </geometry>
         <material name="lidar_orange" />
       </visual>
       <collision>
-        <origin xyz="0.02 0 -0.16" rpy="0 0 0" />
-        <geometry>
-          <box size="0.07 0.05 0.32" />
+        <origin xyz="0.02 0 -0.15" rpy="0 0 0" />
+        <geometry>
+          <box size="0.06 0.045 0.30" />
         </geometry>
       </collision>
       <inertial>
-        <origin xyz="0.02 0 -0.16" rpy="0 0 0" />
+        <origin xyz="0.02 0 -0.15" rpy="0 0 0" />
         <mass value="0.7" />
         <inertia ixx="0.002" ixy="0.0" ixz="0.0" iyy="0.002" iyz="0.0" izz="0.001" />
@@ -303,9 +328,9 @@
       <parent link="torso_link" />
       <child link="${prefix}_arm_link" />
-      <origin xyz="0.0 ${y_offset} ${torso_h - 0.04}" rpy="0 0 0" />
+      <origin xyz="0.0 ${y_offset} ${torso_height - 0.04}" rpy="0 0 0" />
     </joint>
   </xacro:macro>
-  <xacro:arm prefix="left" y_offset="${torso_w/2.0 + 0.025}" />
-  <xacro:arm prefix="right" y_offset="${-torso_w/2.0 - 0.025}" />
+  <xacro:arm prefix="left" y_offset="${torso_width/2.0 + 0.022}" />
+  <xacro:arm prefix="right" y_offset="${-torso_width/2.0 - 0.022}" />
   <!-- ======================================================================== -->
   <!-- IMU Link                                                                 -->
