Commit message: release(v0.0.2): autonomous multi-room navigation, turtlebot3 waffle physics base & spatial mission planner

File: ros2_ws/src/gracemo_description/urdf/gracemo_vira.urdf.xacro (robot description, xacro)
@@ -1,314 +1,317 @@
-<?xml version="1.0"?>
-<robot name="gracemo_vira" xmlns:xacro="http://www.ros.org/wiki/xacro">
-  <!-- Include sub-files -->
-  <xacro:include filename="$(find gracemo_description)/urdf/materials.xacro" />
-  <xacro:include filename="$(find gracemo_description)/urdf/gazebo_plugins.xacro" />
-  <!-- Dimensions & Constants -->
-  <xacro:property name="wheel_radius" value="0.065" />
-  <xacro:property name="wheel_width" value="0.030" />
-  <xacro:property name="wheelbase" value="0.34" />
-  <xacro:property name="chassis_radius" value="0.19" />
-  <xacro:property name="chassis_height" value="0.14" />
-  <xacro:property name="torso_height" value="0.40" />
-  <xacro:property name="torso_width" value="0.20" />
-  <xacro:property name="torso_depth" value="0.16" />
+<?xml version="1.0" ?>
+<!-- ============================================================================== -->
+<!-- GRaCEmo ViRa — Built on Industry-Standard TurtleBot3 Waffle Architecture       -->
+<!-- Factory-Calibrated Physics, Balanced Inertia, Zero-Friction Caster Dynamics   -->
+<!-- ============================================================================== -->
+<robot name="gracemo_vira" xmlns:xacro="http://ros.org/wiki/xacro">
+  <!-- Material Colors -->
+  <material name="black">
+    <color rgba="0.0 0.0 0.0 1.0"/>
+  </material>
+  <material name="dark">
+    <color rgba="0.2 0.2 0.2 1.0"/>
+  </material>
+  <material name="light_black">
+    <color rgba="0.3 0.3 0.3 1.0"/>
+  </material>
+  <material name="chassis_blue">
+    <color rgba="0.0 0.6 0.9 1.0"/>
+  </material>
+  <material name="white">
+    <color rgba="1.0 1.0 1.0 1.0"/>
+  </material>
   <!-- Base Footprint (Ground Projection) -->
-  <link name="base_footprint" />
-  <joint name="base_footprint_joint" type="fixed">
-    <parent link="base_footprint" />
+  <link name="base_footprint"/>
+  <joint name="base_joint" type="fixed">
+    <parent link="base_footprint"/>
     <child link="base_link" />
-    <origin xyz="0 0 ${wheel_radius}" rpy="0 0 0" />
-  </joint>
+    <origin xyz="0 0 0.010" rpy="0 0 0"/>
+  </joint>
+  <!-- Base Link (Chassis) -->
+  <link name="base_link">
+    <visual>
+      <origin xyz="-0.064 0 0.0" rpy="0 0 0"/>
+      <geometry>
+        <mesh filename="package://turtlebot3_description/meshes/bases/waffle_base.stl" scale="0.001 0.001 0.001"/>
+      </geometry>
+      <material name="chassis_blue"/>
+    </visual>
+    <collision>
+      <origin xyz="-0.064 0 0.047" rpy="0 0 0"/>
+      <geometry>
+        <box size="0.266 0.266 0.094"/>
+      </geometry>
+    </collision>
+    <inertial>
+      <origin xyz="0 0 0" rpy="0 0 0"/>
+      <mass value="1.3729096"/>
+      <inertia ixx="8.7002718e-03" ixy="-4.7576583e-05" ixz="1.1160499e-04"
+               iyy="8.6195418e-03" iyz="-3.5422299e-06"
+               izz="1.4612727e-02" />
+    </inertial>
+  </link>
+  <!-- Left Drive Wheel -->
+  <joint name="wheel_left_joint" type="continuous">
+    <parent link="base_link"/>
+    <child link="wheel_left_link"/>
+    <origin xyz="0.0 0.144 0.023" rpy="-1.57 0 0"/>
+    <axis xyz="0 0 1"/>
+  </joint>
+  <link name="wheel_left_link">
+    <visual>
+      <origin xyz="0 0 0" rpy="1.57 0 0"/>
+      <geometry>
+        <mesh filename="package://turtlebot3_description/meshes/wheels/left_tire.stl" scale="0.001 0.001 0.001"/>
+      </geometry>
+      <material name="dark"/>
+    </visual>
+    <collision>
+      <origin xyz="0 0 0" rpy="0 0 0"/>
+      <geometry>
+        <cylinder length="0.018" radius="0.033"/>
+      </geometry>
+    </collision>
+    <inertial>
+      <origin xyz="0 0 0" />
+      <mass value="0.02849894" />
+      <inertia ixx="1.1175580e-05" ixy="-4.2369783e-11" ixz="-5.9381719e-09"
+               iyy="1.1192413e-05" iyz="-1.4400107e-11"
+               izz="2.0712558e-05" />
+    </inertial>
+  </link>
+  <gazebo reference="wheel_left_link">
+    <mu1>1.5</mu1>
+    <mu2>1.5</mu2>
+    <kp>500000.0</kp>
+    <kd>10.0</kd>
+    <minDepth>0.001</minDepth>
+    <maxVel>1.0</maxVel>
+    <material>Gazebo/DarkGrey</material>
+  </gazebo>
+  <!-- Right Drive Wheel -->
+  <joint name="wheel_right_joint" type="continuous">
+    <parent link="base_link"/>
+    <child link="wheel_right_link"/>
+    <origin xyz="0.0 -0.144 0.023" rpy="-1.57 0 0"/>
+    <axis xyz="0 0 1"/>
+  </joint>
+  <link name="wheel_right_link">
+    <visual>
+      <origin xyz="0 0 0" rpy="1.57 0 0"/>
+      <geometry>
+        <mesh filename="package://turtlebot3_description/meshes/wheels/right_tire.stl" scale="0.001 0.001 0.001"/>
+      </geometry>
+      <material name="dark"/>
+    </visual>
+    <collision>
+      <origin xyz="0 0 0" rpy="0 0 0"/>
+      <geometry>
+        <cylinder length="0.018" radius="0.033"/>
+      </geometry>
+    </collision>
+    <inertial>
+      <origin xyz="0 0 0" />
+      <mass value="0.02849894" />
+      <inertia ixx="1.1175580e-05" ixy="-4.2369783e-11" ixz="-5.9381719e-09"
+               iyy="1.1192413e-05" iyz="-1.4400107e-11"
+               izz="2.0712558e-05" />
+    </inertial>
+  </link>
+  <gazebo reference="wheel_right_link">
+    <mu1>1.5</mu1>
+    <mu2>1.5</mu2>
+    <kp>500000.0</kp>
+    <kd>10.0</kd>
+    <minDepth>0.001</minDepth>
+    <maxVel>1.0</maxVel>
+    <material>Gazebo/DarkGrey</material>
+  </gazebo>
+  <!-- Rear Right Caster (Frictionless ball glider) -->
+  <joint name="caster_back_right_joint" type="fixed">
+    <parent link="base_link"/>
+    <child link="caster_back_right_link"/>
+    <origin xyz="-0.177 -0.064 -0.004" rpy="-1.57 0 0"/>
+  </joint>
+  <link name="caster_back_right_link">
+    <collision>
+      <origin xyz="0 0.001 0" rpy="0 0 0"/>
+      <geometry>
+        <sphere radius="0.005"/>
+      </geometry>
+    </collision>
+    <inertial>
+      <origin xyz="0 0 0" />
+      <mass value="0.005" />
+      <inertia ixx="0.00001" ixy="0.0" ixz="0.0" iyy="0.00001" iyz="0.0" izz="0.00001" />
+    </inertial>
+  </link>
+  <gazebo reference="caster_back_right_joint">
+    <preserveFixedJoint>true</preserveFixedJoint>
+  </gazebo>
+  <gazebo reference="caster_back_right_link">
+    <mu1>0.0</mu1>
+    <mu2>0.0</mu2>
+    <kp>100000.0</kp>
+    <kd>1.0</kd>
+    <minDepth>0.001</minDepth>
+    <material>Gazebo/Grey</material>
+  </gazebo>
+  <!-- Rear Left Caster (Frictionless ball glider) -->
+  <joint name="caster_back_left_joint" type="fixed">
+    <parent link="base_link"/>
+    <child link="caster_back_left_link"/>
+    <origin xyz="-0.177 0.064 -0.004" rpy="-1.57 0 0"/>
+  </joint>
+  <link name="caster_back_left_link">
+    <collision>
+      <origin xyz="0 0.001 0" rpy="0 0 0"/>
+      <geometry>
+        <sphere radius="0.005"/>
+      </geometry>
+    </collision>
+    <inertial>
+      <origin xyz="0 0 0" />
+      <mass value="0.005" />
+      <inertia ixx="0.00001" ixy="0.0" ixz="0.0" iyy="0.00001" iyz="0.0" izz="0.00001" />
+    </inertial>
+  </link>
+  <gazebo reference="caster_back_left_joint">
+    <preserveFixedJoint>true</preserveFixedJoint>
+  </gazebo>
+  <gazebo reference="caster_back_left_link">
+    <mu1>0.0</mu1>
+    <mu2>0.0</mu2>
+    <kp>100000.0</kp>
+    <kd>1.0</kd>
+    <minDepth>0.001</minDepth>
+    <material>Gazebo/Grey</material>
+  </gazebo>
+  <!-- 2D RPLiDAR (360-Degree Scan) -->
+  <joint name="scan_joint" type="fixed">
+    <parent link="base_link"/>
+    <child link="base_scan"/>
+    <origin xyz="-0.064 0 0.122" rpy="0 0 0"/>
+  </joint>
+  <link name="base_scan">
+    <visual>
+      <origin xyz="0 0 0.0" rpy="0 0 0"/>
+      <geometry>
+        <mesh filename="package://turtlebot3_description/meshes/sensors/lds.stl" scale="0.001 0.001 0.001"/>
+      </geometry>
+      <material name="dark"/>
+    </visual>
+    <collision>
+      <origin xyz="0.015 0 -0.0065" rpy="0 0 0"/>
+      <geometry>
+        <cylinder length="0.0315" radius="0.055"/>
+      </geometry>
+    </collision>
+    <inertial>
+      <mass value="0.114" />
+      <origin xyz="0 0 0" />
+      <inertia ixx="0.001" ixy="0.0" ixz="0.0" iyy="0.001" iyz="0.0" izz="0.001" />
+    </inertial>
+  </link>
+  <!-- Front RGB Camera -->
+  <joint name="camera_joint" type="fixed">
+    <parent link="base_link"/>
+    <child link="camera_link"/>
+    <origin xyz="0.064 -0.065 0.094" rpy="0 0 0"/>
+  </joint>
+  <link name="camera_link">
+    <visual>
+      <origin xyz="0 0 0" rpy="1.57 0 1.57"/>
+      <geometry>
+        <mesh filename="package://turtlebot3_description/meshes/sensors/r200.dae" />
+      </geometry>
+    </visual>
+    <collision>
+      <origin xyz="0.003 0.065 0.007" rpy="0 0 0"/>
+      <geometry>
+        <box size="0.012 0.132 0.020"/>
+      </geometry>
+    </collision>
+  </link>
+  <joint name="camera_rgb_joint" type="fixed">
+    <parent link="camera_link"/>
+    <child link="camera_rgb_frame"/>
+    <origin xyz="0.005 0.018 0.013" rpy="0 0 0"/>
+  </joint>
+  <link name="camera_rgb_frame"/>
+  <joint name="camera_rgb_optical_joint" type="fixed">
+    <parent link="camera_rgb_frame"/>
+    <child link="camera_rgb_optical_frame"/>
+    <origin xyz="0 0 0" rpy="-1.57 0 -1.57"/>
+  </joint>
+  <link name="camera_rgb_optical_frame"/>
   <!-- ======================================================================== -->
-  <!-- Base Link (Sleek Mobile Chassis with Non-Overlapping Collision)          -->
+  <!-- Gazebo Harmonic 8 Simulation Plugins                                     -->
   <!-- ======================================================================== -->
-  <link name="base_link">
-    <!-- Visual Shell -->
-    <visual>
-      <origin xyz="0 0 ${chassis_height/2.0}" rpy="0 0 0" />
-      <geometry>
-        <cylinder radius="${chassis_radius}" length="${chassis_height}" />
-      </geometry>
-      <material name="chassis_blue" />
-    </visual>
-    <!-- Lower Protective Skirt -->
-    <visual>
-      <origin xyz="0 0 ${chassis_height * 0.2}" rpy="0 0 0" />
-      <geometry>
-        <cylinder radius="${chassis_radius + 0.005}" length="${chassis_height * 0.35}" />
-      </geometry>
-      <material name="dark_grey" />
-    </visual>
-    <!-- Top Deck Plate -->
-    <visual>
-      <origin xyz="0 0 ${chassis_height + 0.005}" rpy="0 0 0" />
-      <geometry>
-        <cylinder radius="${chassis_radius * 0.9}" length="0.01" />
-      </geometry>
-      <material name="dark_grey" />
-    </visual>
-    <collision>
-      <origin xyz="0 0 ${chassis_height/2.0 + 0.01}" rpy="0 0 0" />
-      <geometry>
-        <box size="0.24 0.20 ${chassis_height}" />
-      </geometry>
-    </collision>
-    <!-- Heavy low base mass to keep wheels firmly planted with high traction -->
-    <inertial>
-      <origin xyz="0 0 0.02" rpy="0 0 0" />
-      <mass value="8.0" />
-      <inertia ixx="0.04" ixy="0.0" ixz="0.0" iyy="0.04" iyz="0.0" izz="0.06" />
-    </inertial>
-  </link>
-  <!-- ======================================================================== -->
-  <!-- Drive Wheels (High Grip & Smooth Rolling)                                -->
-  <!-- ======================================================================== -->
-  <xacro:macro name="wheel" params="prefix y_offset">
-    <link name="${prefix}_wheel_link">
-      <visual>
-        <origin xyz="0 0 0" rpy="${pi/2} 0 0" />
-        <geometry>
-          <cylinder radius="${wheel_radius}" length="${wheel_width}" />
-        </geometry>
-        <material name="rubber_black" />
-      </visual>
-      <visual>
-        <origin xyz="0 0 0" rpy="${pi/2} 0 0" />
-        <geometry>
-          <cylinder radius="${wheel_radius * 0.6}" length="${wheel_width + 0.002}" />
-        </geometry>
-        <material name="metallic_silver" />
-      </visual>
-      <collision>
-        <origin xyz="0 0 0" rpy="${pi/2} 0 0" />
-        <geometry>
-          <cylinder radius="${wheel_radius}" length="${wheel_width}" />
-        </geometry>
-      </collision>
-      <inertial>
-        <mass value="0.8" />
-        <inertia ixx="0.001" ixy="0.0" ixz="0.0" iyy="0.001" iyz="0.0" izz="0.001" />
-      </inertial>
-    </link>
-    <joint name="${prefix}_wheel_joint" type="continuous">
-      <parent link="base_link" />
-      <child link="${prefix}_wheel_link" />
-      <origin xyz="0 ${y_offset} 0" rpy="0 0 0" />
-      <axis xyz="0 1 0" />
-      <limit effort="150.0" velocity="20.0" />
-      <dynamics damping="0.01" friction="0.01" />
-    </joint>
-    <gazebo reference="${prefix}_wheel_link">
-      <mu1>1.5</mu1>
-      <mu2>1.5</mu2>
-      <kp>1000000.0</kp>
-      <kd>100.0</kd>
-      <minDepth>0.001</minDepth>
-      <material>Gazebo/DarkGrey</material>
-    </gazebo>
-  </xacro:macro>
-  <xacro:wheel prefix="left" y_offset="${wheelbase/2.0}" />
-  <xacro:wheel prefix="right" y_offset="${-wheelbase/2.0}" />
-  <!-- ======================================================================== -->
-  <!-- Support Casters (Exact ground tangent frictionless gliders)              -->
-  <!-- ======================================================================== -->
-  <xacro:macro name="caster" params="prefix x_offset">
-    <link name="${prefix}_caster_link">
-      <visual>
-        <geometry>
-          <sphere radius="0.025" />
-        </geometry>
-        <material name="metallic_silver" />
-      </visual>
-      <collision>
-        <geometry>
-          <sphere radius="0.025" />
-        </geometry>
-      </collision>
-      <inertial>
-        <mass value="0.05" />
-        <inertia ixx="0.00001" ixy="0.0" ixz="0.0" iyy="0.00001" iyz="0.0" izz="0.00001" />
-      </inertial>
-    </link>
-    <joint name="${prefix}_caster_joint" type="fixed">
-      <parent link="base_link" />
-      <child link="${prefix}_caster_link" />
-      <origin xyz="${x_offset} 0 ${-wheel_radius + 0.027}" rpy="0 0 0" />
-    </joint>
-    <gazebo reference="${prefix}_caster_link">
-      <mu1>0.0</mu1>
-      <mu2>0.0</mu2>
-      <kp>1000.0</kp>
-      <kd>0.1</kd>
-      <minDepth>0.0001</minDepth>
-      <material>Gazebo/Grey</material>
-    </gazebo>
-  </xacro:macro>
-  <xacro:caster prefix="front" x_offset="0.14" />
-  <xacro:caster prefix="rear" x_offset="-0.14" />
-  <!-- ======================================================================== -->
-  <!-- Humanoid Torso (Visual Only — Collision handled by unified base)         -->
-  <!-- ======================================================================== -->
-  <link name="torso_link">
-    <visual>
-      <origin xyz="0 0 ${torso_height/2.0}" rpy="0 0 0" />
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