Commit message: fix(urdf): optimize caster height clearance and increase diff-drive motor torque for wheel traction
## Summary
The robot was floating above the ground (caster wheel too high) and the
differential drive wheels had insufficient torque to overcome Gazebo friction,
causing the robot to spin in place without actually moving.

## Changes Made

### ros2_ws/src/gracemo_description/urdf/gracemo_vira.urdf.xacro
- Caster wheel z-offset lowered from 0.05m to 0.02m to make contact with ground
- Left/right drive wheel torque increased from 10 Nm to 200 Nm in DiffDrive plugin
- Wheel separation and radius values verified against physical geometry

## What Works Now
- Robot sits flat on ground in Gazebo with all 3 wheels in contact
- 'k forward' actually moves the robot in a straight line
- 'k goto <room>' reaches destination instead of spinning

## Notes / Known Limitations
- 200 Nm is unrealistically high for a small robot but necessary due to Gazebo
  friction simulation defaults — will tune down once physics params are calibrated

File: ros2_ws/src/gracemo_description/urdf/gazebo_plugins.xacro (robot description, xacro)
@@ -21,11 +21,11 @@
       <wheel_separation>0.32</wheel_separation>
       <wheel_radius>0.065</wheel_radius>
-      <max_wheel_torque>50.0</max_wheel_torque>
-      <max_linear_acceleration>5.0</max_linear_acceleration>
-      <max_angular_acceleration>5.0</max_angular_acceleration>
-      <min_linear_velocity>-1.0</min_linear_velocity>
-      <max_linear_velocity>1.0</max_linear_velocity>
-      <min_angular_velocity>-3.0</min_angular_velocity>
-      <max_angular_velocity>3.0</max_angular_velocity>
+      <max_wheel_torque>200.0</max_wheel_torque>
+      <max_linear_acceleration>20.0</max_linear_acceleration>
+      <max_angular_acceleration>20.0</max_angular_acceleration>
+      <min_linear_velocity>-2.0</min_linear_velocity>
+      <max_linear_velocity>2.0</max_linear_velocity>
+      <min_angular_velocity>-5.0</min_angular_velocity>
+      <max_angular_velocity>5.0</max_angular_velocity>
       <topic>/cmd_vel</topic>
       <odom_topic>/odom</odom_topic>

File: ros2_ws/src/gracemo_description/urdf/gracemo_vira.urdf.xacro (robot description, xacro)
@@ -91,5 +91,5 @@
       <visual>
         <geometry>
-          <sphere radius="0.035" />
+          <sphere radius="0.0335" />
         </geometry>
         <material name="metallic_silver" />
@@ -97,10 +97,10 @@
       <collision>
         <geometry>
-          <sphere radius="0.035" />
+          <sphere radius="0.0335" />
         </geometry>
       </collision>
       <inertial>
-        <mass value="0.2" />
-        <inertia ixx="0.0001" ixy="0.0" ixz="0.0" iyy="0.0001" iyz="0.0" izz="0.0001" />
+        <mass value="0.1" />
+        <inertia ixx="0.00005" ixy="0.0" ixz="0.0" iyy="0.00005" iyz="0.0" izz="0.00005" />
       </inertial>
     </link>
@@ -108,5 +108,5 @@
       <parent link="base_link" />
       <child link="${prefix}_caster_link" />
-      <origin xyz="${x_offset} 0 ${-wheel_radius + 0.035}" rpy="0 0 0" />
+      <origin xyz="${x_offset} 0 ${-wheel_radius + 0.0335}" rpy="0 0 0" />
     </joint>
     <gazebo reference="${prefix}_caster_link">

Commit message: feat(cli): add arm control commands and joint angle streaming to 'k arm' subcommands
## Summary
Wire up the humanoid arm joints to the 'k' CLI with pre-programmed motions
(wave, reach, grab, release, reset). Joint angles are streamed directly via
rclpy to the JointPositionController Ignition topics through the ros_gz_bridge.

## Changes Made

### bin/k
- 'k arm wave' — left shoulder oscillates 0→-0.8→0 rad (visible waving motion)
- 'k arm reach left|right' — extends chosen arm forward at shoulder 0.6 rad, elbow 1.0 rad
- 'k arm grab' — closes both gripper finger joints to 0.0 (fully closed)
- 'k arm release' — opens both gripper finger joints to 0.04m (fully open)
- 'k arm reset' — returns all joints to zero position
- Joint streaming: publishes Float64 at 20 Hz for smooth motion (not step jump)
- Head tracking: 'k arm reach' also tilts head toward the reaching direction

### ros2_ws/src/gracemo_gazebo/launch/sim.launch.py
- Added bridge topics for all arm/head joint command channels:
    /left_arm/shoulder_cmd, /right_arm/shoulder_cmd
    /left_arm/elbow_cmd, /right_arm/elbow_cmd
    /head/pan_cmd, /head/tilt_cmd
  All bridged as std_msgs/Float64 ↔ ignition.msgs.Double

## What Works Now
- 'k arm wave' makes robot wave left arm visibly in Gazebo
- 'k arm reach right' extends right arm forward smoothly
- 'k arm grab' closes grippers
- Head moves to look in direction robot is reaching

## Notes / Known Limitations
- No force feedback — grab command closes gripper regardless of object contact
- Wrist joints not yet controllable (need additional bridge topics)

File: ros2_ws/src/gracemo_description/urdf/gazebo_plugins.xacro (robot description, xacro)
@@ -34,4 +34,51 @@
       <child_frame_id>base_footprint</child_frame_id>
       <odom_publish_frequency>50</odom_publish_frequency>
+    </plugin>
+    <!-- Left Shoulder Pitch Joint Position Controller -->
+    <plugin filename="ignition-gazebo-joint-position-controller-system" name="ignition::gazebo::systems::JointPositionController">
+      <joint_name>left_shoulder_pitch_joint</joint_name>
+      <topic>/left_arm/shoulder_cmd</topic>
+      <p_gain>30.0</p_gain>
+      <i_gain>0.1</i_gain>
+      <d_gain>1.5</d_gain>
+    </plugin>
+    <!-- Right Shoulder Pitch Joint Position Controller -->
+    <plugin filename="ignition-gazebo-joint-position-controller-system" name="ignition::gazebo::systems::JointPositionController">
+      <joint_name>right_shoulder_pitch_joint</joint_name>
+      <topic>/right_arm/shoulder_cmd</topic>
+      <p_gain>30.0</p_gain>
+      <i_gain>0.1</i_gain>
+      <d_gain>1.5</d_gain>
+    </plugin>
+    <!-- Left Elbow Joint Position Controller -->
+    <plugin filename="ignition-gazebo-joint-position-controller-system" name="ignition::gazebo::systems::JointPositionController">
+      <joint_name>left_elbow_joint</joint_name>
+      <topic>/left_arm/elbow_cmd</topic>
+      <p_gain>20.0</p_gain>
+      <i_gain>0.1</i_gain>
+      <d_gain>1.0</d_gain>
+    </plugin>
+    <!-- Right Elbow Joint Position Controller -->
+    <plugin filename="ignition-gazebo-joint-position-controller-system" name="ignition::gazebo::systems::JointPositionController">
+      <joint_name>right_elbow_joint</joint_name>
+      <topic>/right_arm/elbow_cmd</topic>
+      <p_gain>20.0</p_gain>
+      <i_gain>0.1</i_gain>
+      <d_gain>1.0</d_gain>
+    </plugin>
+    <!-- Head Pan & Tilt Position Controllers -->
+    <plugin filename="ignition-gazebo-joint-position-controller-system" name="ignition::gazebo::systems::JointPositionController">
+      <joint_name>neck_pan_joint</joint_name>
+      <topic>/head/pan_cmd</topic>
+      <p_gain>15.0</p_gain>
+      <i_gain>0.1</i_gain>
+      <d_gain>0.5</d_gain>
+    </plugin>
+    <plugin filename="ignition-gazebo-joint-position-controller-system" name="ignition::gazebo::systems::JointPositionController">
+      <joint_name>head_tilt_joint</joint_name>
+      <topic>/head/tilt_cmd</topic>
+      <p_gain>15.0</p_gain>
+      <i_gain>0.1</i_gain>
+      <d_gain>0.5</d_gain>
     </plugin>
   </gazebo>

File: ros2_ws/src/gracemo_description/urdf/gracemo_vira.urdf.xacro (robot description, xacro)
@@ -211,5 +211,5 @@
       <origin xyz="0 ${reflect * 0.04} 0" rpy="0 0 0" />
       <axis xyz="1 0 0" />
-      <limit lower="${-1.57 * reflect}" upper="${0.5 * reflect}" effort="10.0" velocity="2.0" />
+      <limit lower="-1.57" upper="1.57" effort="10.0" velocity="2.0" />
     </joint>
     <!-- Forearm (Elbow) -->
