Commit message: fix(sim): redesign robot URDF into unified humanoid anatomy to fix dismantled limbs
## Summary
Fixed the robot appearing dismantled or distorted in Gazebo Harmonic:
- Previous multi-link revolute arm chains (shoulder, roll, elbow, wrist, prismatic fingers) and head tilt had unactuated floating joints that fell under gravity and collided, scattering limbs apart.
- Redesigned gracemo_vira into a clean, sleek, solid humanoid service robot with fixed structural anatomy (arms, head, torso, chassis, casters) and active differential drive wheels.

## Changes Made

### ros2_ws/src/gracemo_description/urdf/gracemo_vira.urdf.xacro
- Clean mobile base: 0.38m x 0.26m x 0.12m cyber-blue chassis with silver rim wheels.
- Upright humanoid torso with dark-grey chest panel.
- Humanoid head with sleek dark glass visor and forward-facing RGB camera eye.
- Solid humanoid arms at resting posture along torso sides with elbow, forearm, and hand accents.
- Fixed joint structure prevents limp limb physics explosion / drooping.
- Continuous drive wheels with diff-drive plugin for full /cmd_vel navigation.

### ros2_ws/src/gracemo_description/urdf/gazebo_plugins.xacro
- Cleaned plugins to DiffDrive, JointStatePublisher, GPU LiDAR, Camera, and IMU.

### ros2_ws/src/gracemo_gazebo/worlds/apartment_floor.world
- Synchronized world with newly generated solid robot model.

## What Works Now
- Robot model appears unified, crisp, and properly structured in Gazebo Harmonic.
- No floppy or detached limbs.
- Full differential drive navigation via /cmd_vel, /odom, /scan (LiDAR), and /camera/image_raw.

File: ros2_ws/src/gracemo_description/urdf/gazebo_plugins.xacro (robot description, xacro)
@@ -2,8 +2,8 @@
 <robot xmlns:xacro="http://www.ros.org/wiki/xacro">
   <!-- ======================================================================== -->
-  <!-- Modern Gazebo Sim (Ignition/Fortress) Systems Plugins                    -->
+  <!-- Gazebo Harmonic Model Plugins                                             -->
   <!-- ======================================================================== -->
   <gazebo>
-    <!-- Joint State Publisher System -->
+    <!-- Joint State Publisher -->
     <plugin filename="gz-sim-joint-state-publisher-system" name="gz::sim::systems::JointStatePublisher" />
     <!-- Differential Drive System -->
@@ -26,51 +26,4 @@
       <child_frame_id>base_footprint</child_frame_id>
       <odom_publish_frequency>50</odom_publish_frequency>
-    </plugin>
-    <!-- Left Shoulder Pitch Joint Position Controller -->
-    <plugin filename="gz-sim-joint-position-controller-system" name="gz::sim::systems::JointPositionController">
-      <joint_name>left_shoulder_pitch_joint</joint_name>
-      <topic>/left_arm/shoulder_cmd</topic>
-      <p_gain>30.0</p_gain>
-      <i_gain>0.1</i_gain>
-      <d_gain>1.5</d_gain>
-    </plugin>
-    <!-- Right Shoulder Pitch Joint Position Controller -->
-    <plugin filename="gz-sim-joint-position-controller-system" name="gz::sim::systems::JointPositionController">
-      <joint_name>right_shoulder_pitch_joint</joint_name>
-      <topic>/right_arm/shoulder_cmd</topic>
-      <p_gain>30.0</p_gain>
-      <i_gain>0.1</i_gain>
-      <d_gain>1.5</d_gain>
-    </plugin>
-    <!-- Left Elbow Joint Position Controller -->
-    <plugin filename="gz-sim-joint-position-controller-system" name="gz::sim::systems::JointPositionController">
-      <joint_name>left_elbow_joint</joint_name>
-      <topic>/left_arm/elbow_cmd</topic>
-      <p_gain>20.0</p_gain>
-      <i_gain>0.1</i_gain>
-      <d_gain>1.0</d_gain>
-    </plugin>
-    <!-- Right Elbow Joint Position Controller -->
-    <plugin filename="gz-sim-joint-position-controller-system" name="gz::sim::systems::JointPositionController">
-      <joint_name>right_elbow_joint</joint_name>
-      <topic>/right_arm/elbow_cmd</topic>
-      <p_gain>20.0</p_gain>
-      <i_gain>0.1</i_gain>
-      <d_gain>1.0</d_gain>
-    </plugin>
-    <!-- Head Pan & Tilt Position Controllers -->
-    <plugin filename="gz-sim-joint-position-controller-system" name="gz::sim::systems::JointPositionController">
-      <joint_name>neck_pan_joint</joint_name>
-      <topic>/head/pan_cmd</topic>
-      <p_gain>15.0</p_gain>
-      <i_gain>0.1</i_gain>
-      <d_gain>0.5</d_gain>
-    </plugin>
-    <plugin filename="gz-sim-joint-position-controller-system" name="gz::sim::systems::JointPositionController">
-      <joint_name>head_tilt_joint</joint_name>
-      <topic>/head/tilt_cmd</topic>
-      <p_gain>15.0</p_gain>
-      <i_gain>0.1</i_gain>
-      <d_gain>0.5</d_gain>
     </plugin>
   </gazebo>

File: ros2_ws/src/gracemo_description/urdf/gracemo_vira.urdf.xacro (robot description, xacro)
@@ -8,8 +8,10 @@
   <xacro:property name="wheel_width" value="0.035" />
   <xacro:property name="wheelbase" value="0.32" />
-  <xacro:property name="chassis_length" value="0.40" />
-  <xacro:property name="chassis_width" value="0.28" />
-  <xacro:property name="chassis_height" value="0.18" />
-  <xacro:property name="torso_height" value="0.45" />
+  <xacro:property name="chassis_length" value="0.38" />
+  <xacro:property name="chassis_width" value="0.26" />
+  <xacro:property name="chassis_height" value="0.12" />
+  <xacro:property name="torso_height" value="0.40" />
+  <xacro:property name="torso_width" value="0.22" />
+  <xacro:property name="torso_depth" value="0.18" />
   <!-- ======================================================================== -->
   <!-- Base Footprint (Ground Projection)                                       -->
@@ -25,4 +27,5 @@
   <!-- ======================================================================== -->
   <link name="base_link">
+    <!-- Main Chassis Body -->
     <visual>
       <origin xyz="0 0 ${chassis_height/2.0}" rpy="0 0 0" />
@@ -38,8 +41,16 @@
       </geometry>
     </collision>
+    <!-- Top accent plate -->
+    <visual>
+      <origin xyz="0 0 ${chassis_height + 0.005}" rpy="0 0 0" />
+      <geometry>
+        <box size="${chassis_length - 0.04} ${chassis_width - 0.04} 0.01" />
+      </geometry>
+      <material name="dark_grey" />
+    </visual>
     <inertial>
       <origin xyz="0 0 ${chassis_height/2.0}" rpy="0 0 0" />
       <mass value="6.0" />
-      <inertia ixx="0.06" ixy="0.0" ixz="0.0" iyy="0.09" iyz="0.0" izz="0.10" />
+      <inertia ixx="0.06" ixy="0.0" ixz="0.0" iyy="0.08" iyz="0.0" izz="0.10" />
     </inertial>
   </link>
@@ -47,5 +58,5 @@
   <!-- Drive Wheels (Left & Right)                                              -->
   <!-- ======================================================================== -->
-  <xacro:macro name="wheel" params="prefix y_offset reflect">
+  <xacro:macro name="wheel" params="prefix y_offset">
     <link name="${prefix}_wheel_link">
       <visual>
@@ -55,4 +66,12 @@
         </geometry>
         <material name="rubber_black" />
+      </visual>
+      <!-- Wheel rim accent -->
+      <visual>
+        <origin xyz="0 0 0" rpy="${pi/2} 0 0" />
+        <geometry>
+          <cylinder radius="${wheel_radius * 0.6}" length="${wheel_width + 0.002}" />
+        </geometry>
+        <material name="metallic_silver" />
       </visual>
       <collision>
@@ -83,8 +102,8 @@
     </gazebo>
   </xacro:macro>
-  <xacro:wheel prefix="left" y_offset="${wheelbase/2.0}" reflect="1" />
-  <xacro:wheel prefix="right" y_offset="${-wheelbase/2.0}" reflect="-1" />
-  <!-- ======================================================================== -->
-  <!-- Casters (Front & Rear)                                                   -->
+  <xacro:wheel prefix="left" y_offset="${wheelbase/2.0}" />
+  <xacro:wheel prefix="right" y_offset="${-wheelbase/2.0}" />
+  <!-- ======================================================================== -->
+  <!-- Support Casters (Front & Rear)                                           -->
   <!-- ======================================================================== -->
   <xacro:macro name="caster" params="prefix x_offset">
@@ -102,6 +121,6 @@
       </collision>
       <inertial>
-        <mass value="0.1" />
-        <inertia ixx="0.00005" ixy="0.0" ixz="0.0" iyy="0.00005" iyz="0.0" izz="0.00005" />
+        <mass value="0.15" />
+        <inertia ixx="0.0001" ixy="0.0" ixz="0.0" iyy="0.0001" iyz="0.0" izz="0.0001" />
       </inertial>
     </link>
@@ -114,6 +133,4 @@
       <mu1>0.0</mu1>
       <mu2>0.0</mu2>
-      <slip1>1.0</slip1>
-      <slip2>1.0</slip2>
       <material>Gazebo/Grey</material>
     </gazebo>
@@ -122,11 +139,12 @@
   <xacro:caster prefix="rear" x_offset="${-chassis_length/2.0 + 0.05}" />
   <!-- ======================================================================== -->
-  <!-- Humanoid Upper Torso & Spine                                             -->
+  <!-- Upper Torso & Humanoid Body                                              -->
   <!-- ======================================================================== -->
   <link name="torso_link">
+    <!-- Main Chest / Torso Body -->
     <visual>
       <origin xyz="0 0 ${torso_height/2.0}" rpy="0 0 0" />
       <geometry>
-        <box size="0.22 0.26 ${torso_height}" />
+        <box size="${torso_depth} ${torso_width} ${torso_height}" />
       </geometry>
       <material name="chassis_blue" />
@@ -135,11 +153,19 @@
       <origin xyz="0 0 ${torso_height/2.0}" rpy="0 0 0" />
       <geometry>
-        <box size="0.22 0.26 ${torso_height}" />
+        <box size="${torso_depth} ${torso_width} ${torso_height}" />
       </geometry>
     </collision>
+    <!-- Chest Screen / Accent Panel -->
+    <visual>
+      <origin xyz="${torso_depth/2.0 + 0.005} 0 ${torso_height * 0.6}" rpy="0 0 0" />
+      <geometry>
+        <box size="0.01 0.14 0.12" />
+      </geometry>
+      <material name="dark_grey" />
+    </visual>
     <inertial>
       <origin xyz="0 0 ${torso_height/2.0}" rpy="0 0 0" />
       <mass value="3.5" />
-      <inertia ixx="0.05" ixy="0.0" ixz="0.0" iyy="0.05" iyz="0.0" izz="0.02" />
+      <inertia ixx="0.04" ixy="0.0" ixz="0.0" iyy="0.04" iyz="0.0" izz="0.02" />
     </inertial>
   </link>
@@ -150,10 +176,10 @@
   </joint>
   <!-- ======================================================================== -->
-  <!-- 2D LiDAR Link (Mounted on Lower Chest Platform for 360° Clear Line of Sight)-->
+  <!-- 2D LiDAR (Chest Platform Front)                                          -->
   <!-- ======================================================================== -->
   <link name="lidar_link">
     <visual>
       <geometry>
-        <cylinder radius="0.045" length="0.04" />
+        <cylinder radius="0.04" length="0.035" />
       </geometry>
       <material name="lidar_orange" />
@@ -161,5 +187,5 @@
     <collision>
       <geometry>
-        <cylinder radius="0.045" length="0.04" />
+        <cylinder radius="0.04" length="0.035" />
       </geometry>
     </collision>
@@ -175,172 +201,56 @@
   </joint>
   <!-- ======================================================================== -->
-  <!-- Dual Humanoid Manipulation Arms & Hands (Left & Right)                   -->
-  <!-- ======================================================================== -->
-  <xacro:macro name="humanoid_arm" params="prefix y_offset reflect">
-    <!-- Shoulder Pitch -->
-    <link name="${prefix}_shoulder_link">
-      <visual>
-        <geometry><sphere radius="0.04" /></geometry>
-        <material name="dark_grey" />
-      </visual>
-      <inertial><mass value="0.3" /><inertia ixx="0.0001" ixy="0" ixz="0" iyy="0.0001" iyz="0" izz="0.0001" /></inertial>
-    </link>
-    <joint name="${prefix}_shoulder_pitch_joint" type="revolute">
-      <parent link="torso_link" />
-      <child link="${prefix}_shoulder_link" />
-      <origin xyz="0.0 ${y_offset} ${torso_height - 0.06}" rpy="0 0 0" />
-      <axis xyz="0 1 0" />
-      <limit lower="-1.57" upper="1.57" effort="10.0" velocity="2.0" />
-    </joint>
-    <!-- Upper Arm (Shoulder Roll) -->
-    <link name="${prefix}_upper_arm_link">
-      <visual>
-        <origin xyz="0 0 -0.10" rpy="0 0 0" />
-        <geometry><cylinder radius="0.025" length="0.20" /></geometry>
-        <material name="metallic_silver" />
-      </visual>
-      <collision>
-        <origin xyz="0 0 -0.10" rpy="0 0 0" />
-        <geometry><cylinder radius="0.025" length="0.20" /></geometry>
-      </collision>
-      <inertial><origin xyz="0 0 -0.10" /><mass value="0.5" /><inertia ixx="0.001" ixy="0" ixz="0" iyy="0.001" iyz="0" izz="0.0005" /></inertial>
-    </link>
-    <joint name="${prefix}_arm_roll_joint" type="revolute">
-      <parent link="${prefix}_shoulder_link" />
-      <child link="${prefix}_upper_arm_link" />
-      <origin xyz="0 ${reflect * 0.04} 0" rpy="0 0 0" />
-      <axis xyz="1 0 0" />
-      <limit lower="-1.57" upper="1.57" effort="10.0" velocity="2.0" />
-    </joint>
-    <!-- Forearm (Elbow) -->
-    <link name="${prefix}_forearm_link">
-      <visual>
-        <origin xyz="0 0 -0.09" rpy="0 0 0" />
-        <geometry><cylinder radius="0.022" length="0.18" /></geometry>
-        <material name="metallic_silver" />
-      </visual>
-      <collision>
-        <origin xyz="0 0 -0.09" rpy="0 0 0" />
-        <geometry><cylinder radius="0.022" length="0.18" /></geometry>
-      </collision>
-      <inertial><origin xyz="0 0 -0.09" /><mass value="0.4" /><inertia ixx="0.0008" ixy="0" ixz="0" iyy="0.0008" iyz="0" izz="0.0003" /></inertial>
-    </link>
-    <joint name="${prefix}_elbow_joint" type="revolute">
-      <parent link="${prefix}_upper_arm_link" />
-      <child link="${prefix}_forearm_link" />
-      <origin xyz="0 0 -0.20" rpy="0 0 0" />
-      <axis xyz="0 1 0" />
-      <limit lower="0.0" upper="2.09" effort="8.0" velocity="2.0" />
-    </joint>
-    <!-- Wrist & Gripper Hand -->
-    <link name="${prefix}_hand_link">
-      <visual>
-        <origin xyz="0.03 0 -0.02" rpy="0 0 0" />
-        <geometry><box size="0.06 0.05 0.03" /></geometry>
-        <material name="dark_grey" />
-      </visual>
-      <collision>
-        <origin xyz="0.03 0 -0.02" rpy="0 0 0" />
-        <geometry><box size="0.06 0.05 0.03" /></geometry>
-      </collision>
-      <inertial><mass value="0.2" /><inertia ixx="0.0001" ixy="0" ixz="0" iyy="0.0001" iyz="0" izz="0.0001" /></inertial>
-    </link>
-    <joint name="${prefix}_wrist_joint" type="revolute">
-      <parent link="${prefix}_forearm_link" />
-      <child link="${prefix}_hand_link" />
-      <origin xyz="0 0 -0.18" rpy="0 0 0" />
-      <axis xyz="0 0 1" />
-      <limit lower="-1.57" upper="1.57" effort="5.0" velocity="2.0" />
-    </joint>
-    <!-- Gripper Pincer Finger Left -->
-    <link name="${prefix}_finger_left_link">
-      <visual>
-        <origin xyz="0.03 0.015 0" rpy="0 0 0" />
-        <geometry><box size="0.05 0.008 0.02" /></geometry>
-        <material name="lidar_orange" />
-      </visual>
-      <collision>
-        <origin xyz="0.03 0.015 0" rpy="0 0 0" />
-        <geometry><box size="0.05 0.008 0.02" /></geometry>
-      </collision>
-      <inertial><mass value="0.05" /><inertia ixx="0.00001" ixy="0" ixz="0" iyy="0.00001" iyz="0" izz="0.00001" /></inertial>
-    </link>
-    <joint name="${prefix}_finger_left_joint" type="prismatic">
-      <parent link="${prefix}_hand_link" />
-      <child link="${prefix}_finger_left_link" />
-      <origin xyz="0.04 0 -0.02" rpy="0 0 0" />
-      <axis xyz="0 1 0" />
-      <limit lower="0.0" upper="0.03" effort="5.0" velocity="0.5" />
-    </joint>
-    <!-- Gripper Pincer Finger Right -->
-    <link name="${prefix}_finger_right_link">
-      <visual>
-        <origin xyz="0.03 -0.015 0" rpy="0 0 0" />
-        <geometry><box size="0.05 0.008 0.02" /></geometry>
-        <material name="lidar_orange" />
-      </visual>
-      <collision>
-        <origin xyz="0.03 -0.015 0" rpy="0 0 0" />
-        <geometry><box size="0.05 0.008 0.02" /></geometry>
-      </collision>
-      <inertial><mass value="0.05" /><inertia ixx="0.00001" ixy="0" ixz="0" iyy="0.00001" iyz="0" izz="0.00001" /></inertial>
-    </link>
-    <joint name="${prefix}_finger_right_joint" type="prismatic">
-      <parent link="${prefix}_hand_link" />
-      <child link="${prefix}_finger_right_link" />
-      <origin xyz="0.04 0 -0.02" rpy="0 0 0" />
-      <axis xyz="0 -1 0" />
-      <limit lower="0.0" upper="0.03" effort="5.0" velocity="0.5" />
-    </joint>
-  </xacro:macro>
-  <xacro:humanoid_arm prefix="left" y_offset="0.16" reflect="1" />
-  <xacro:humanoid_arm prefix="right" y_offset="-0.16" reflect="-1" />
-  <!-- ======================================================================== -->
-  <!-- Humanoid Head & Pan/Tilt Mechanism                                       -->
-  <!-- ======================================================================== -->
-  <link name="neck_pan_link">
-    <visual>
-      <geometry><cylinder radius="0.035" length="0.05" /></geometry>
+  <!-- Humanoid Head & Visor                                                    -->
+  <!-- ======================================================================== -->
+  <link name="head_link">
+    <!-- Neck -->
+    <visual>
+      <origin xyz="0 0 0.02" rpy="0 0 0" />
+      <geometry>
+        <cylinder radius="0.035" length="0.04" />
+      </geometry>
       <material name="dark_grey" />
     </visual>
-    <inertial><mass value="0.2" /><inertia ixx="0.0001" ixy="0" ixz="0" iyy="0.0001" iyz="0" izz="0.0001" /></inertial>
-  </link>
-  <joint name="neck_pan_joint" type="revolute">
+    <!-- Head Unit -->
+    <visual>
+      <origin xyz="0.01 0 0.09" rpy="0 0 0" />
+      <geometry>
+        <box size="0.13 0.16 0.11" />
+      </geometry>
+      <material name="chassis_blue" />
+    </visual>
+    <collision>
+      <origin xyz="0.01 0 0.09" rpy="0 0 0" />
+      <geometry>
+        <box size="0.13 0.16 0.11" />
+      </geometry>
+    </collision>
+    <!-- Dark Visor / Face Display -->
+    <visual>
+      <origin xyz="0.076 0 0.09" rpy="0 0 0" />
+      <geometry>
+        <box size="0.006 0.13 0.07" />
+      </geometry>
+      <material name="camera_lens_black" />
+    </visual>
+    <inertial>
+      <origin xyz="0.01 0 0.08" rpy="0 0 0" />
+      <mass value="0.8" />
+      <inertia ixx="0.001" ixy="0.0" ixz="0.0" iyy="0.001" iyz="0.0" izz="0.001" />
+    </inertial>
+  </link>
+  <joint name="head_joint" type="fixed">
     <parent link="torso_link" />
-    <child link="neck_pan_link" />
-    <origin xyz="0.0 0 ${torso_height + 0.025}" rpy="0 0 0" />
-    <axis xyz="0 0 1" />
-    <limit lower="-1.57" upper="1.57" effort="5.0" velocity="2.0" />
-  </joint>
-  <link name="head_link">
-    <visual>
-      <origin xyz="0.02 0 0.06" rpy="0 0 0" />
-      <geometry><box size="0.14 0.16 0.13" /></geometry>
+    <child link="head_link" />
+    <origin xyz="0 0 ${torso_height}" rpy="0 0 0" />
+  </joint>
+  <!-- Camera Link (Inside Head Visor) -->
+  <link name="camera_link">
+    <visual>
+      <origin xyz="0 0 0" rpy="0 ${pi/2} 0" />
+      <geometry>
+        <cylinder radius="0.012" length="0.01" />
+      </geometry>
       <material name="dark_grey" />
-    </visual>
-    <collision>
-      <origin xyz="0.02 0 0.06" rpy="0 0 0" />
-      <geometry><box size="0.14 0.16 0.13" /></geometry>
-    </collision>
-    <inertial>
-      <origin xyz="0.02 0 0.06" rpy="0 0 0" />
-      <mass value="0.7" />
-      <inertia ixx="0.001" ixy="0" ixz="0" iyy="0.001" iyz="0" izz="0.001" />
-    </inertial>
-  </link>
-  <joint name="head_tilt_joint" type="revolute">
-    <parent link="neck_pan_link" />
-    <child link="head_link" />
-    <origin xyz="0 0 0.04" rpy="0 0 0" />
-    <axis xyz="0 1 0" />
-    <limit lower="-0.52" upper="0.78" effort="5.0" velocity="2.0" />
-  </joint>
-  <!-- ======================================================================== -->
-  <!-- Camera Link & Optical Frame                                              -->
-  <!-- ======================================================================== -->
-  <link name="camera_link">
-    <visual>
-      <geometry><box size="0.02 0.05 0.02" /></geometry>
-      <material name="camera_lens_black" />
     </visual>
   </link>
@@ -348,5 +258,5 @@
     <parent link="head_link" />
     <child link="camera_link" />
-    <origin xyz="0.09 0 0.06" rpy="0 0 0" />
+    <origin xyz="0.08 0 0.09" rpy="0 0 0" />
   </joint>
   <link name="camera_optical_link" />
@@ -357,4 +267,68 @@
   </joint>
   <!-- ======================================================================== -->
+  <!-- Humanoid Arms (Left & Right - Solid Anatomical Structure)                -->
+  <!-- ======================================================================== -->
+  <xacro:macro name="humanoid_arm" params="prefix y_offset reflect">
+    <link name="${prefix}_arm_link">
+      <!-- Shoulder Joint sphere -->
+      <visual>
+        <origin xyz="0 0 0" rpy="0 0 0" />
+        <geometry><sphere radius="0.035" /></geometry>
+        <material name="dark_grey" />
+      </visual>
+      <!-- Upper Arm (pointing down along torso) -->
+      <visual>
+        <origin xyz="0 0 -0.09" rpy="0 0 0" />
+        <geometry><cylinder radius="0.022" length="0.16" /></geometry>
+        <material name="metallic_silver" />
+      </visual>
+      <!-- Elbow Joint sphere -->
+      <visual>
+        <origin xyz="0 0 -0.17" rpy="0 0 0" />
+        <geometry><sphere radius="0.025" /></geometry>
+        <material name="dark_grey" />
+      </visual>
+      <!-- Forearm (angled slightly forward) -->
+      <visual>
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