Commit message: fix(physics): eliminate caster ground contact friction chatter and smooth diff_drive limits
## Summary
- Replaced 200Nm / 20m/s^2 excessive diff_drive acceleration with smooth realistic limits (25Nm / 2.5m/s^2).
- Adjusted caster collision radius and ground clearance to eliminate ground friction chatter and physics micro-bouncing.
- Rebuilt workspace and synchronized apartment_floor.world.

File: ros2_ws/src/gracemo_description/urdf/gazebo_plugins.xacro (robot description, xacro)
@@ -13,11 +13,11 @@
       <wheel_separation>0.32</wheel_separation>
       <wheel_radius>0.065</wheel_radius>
-      <max_wheel_torque>200.0</max_wheel_torque>
-      <max_linear_acceleration>20.0</max_linear_acceleration>
-      <max_angular_acceleration>20.0</max_angular_acceleration>
-      <min_linear_velocity>-2.0</min_linear_velocity>
-      <max_linear_velocity>2.0</max_linear_velocity>
-      <min_angular_velocity>-5.0</min_angular_velocity>
-      <max_angular_velocity>5.0</max_angular_velocity>
+      <max_wheel_torque>25.0</max_wheel_torque>
+      <max_linear_acceleration>2.5</max_linear_acceleration>
+      <max_angular_acceleration>3.5</max_angular_acceleration>
+      <min_linear_velocity>-1.0</min_linear_velocity>
+      <max_linear_velocity>1.0</max_linear_velocity>
+      <min_angular_velocity>-2.5</min_angular_velocity>
+      <max_angular_velocity>2.5</max_angular_velocity>
       <topic>/cmd_vel</topic>
       <odom_topic>/odom</odom_topic>

File: ros2_ws/src/gracemo_description/urdf/gracemo_vira.urdf.xacro (robot description, xacro)
@@ -117,5 +117,5 @@
       <visual>
         <geometry>
-          <sphere radius="0.0335" />
+          <sphere radius="0.032" />
         </geometry>
         <material name="metallic_silver" />
@@ -123,9 +123,9 @@
       <collision>
         <geometry>
-          <sphere radius="0.0335" />
+          <sphere radius="0.030" />
         </geometry>
       </collision>
       <inertial>
-        <mass value="0.15" />
+        <mass value="0.10" />
         <inertia ixx="0.0001" ixy="0.0" ixz="0.0" iyy="0.0001" iyz="0.0" izz="0.0001" />
       </inertial>
@@ -134,9 +134,11 @@
       <parent link="base_link" />
       <child link="${prefix}_caster_link" />
-      <origin xyz="${x_offset} 0 ${-wheel_radius + 0.0335}" rpy="0 0 0" />
+      <origin xyz="${x_offset} 0 ${-wheel_radius + 0.032}" rpy="0 0 0" />
     </joint>
     <gazebo reference="${prefix}_caster_link">
       <mu1>0.0</mu1>
       <mu2>0.0</mu2>
+      <kp>100000.0</kp>
+      <kd>10.0</kd>
       <material>Gazebo/Grey</material>
     </gazebo>

Commit message: fix(physics): fix wheel scrub torque stall and match wheel separation
## Summary
- Fixed wheel torque limit (raised to 150 Nm) and normalized lateral wheel friction (mu1=1.5, mu2=1.5), preventing in-place rotation stall caused by excessive sideways tire scrubbing resistance.
- Synchronized wheel_separation to 0.34m in DiffDrive plugin.
- Rebuilt workspace and updated apartment_floor.world.

File: ros2_ws/src/gracemo_description/urdf/gazebo_plugins.xacro (robot description, xacro)
@@ -11,13 +11,13 @@
       <left_joint>left_wheel_joint</left_joint>
       <right_joint>right_wheel_joint</right_joint>
-      <wheel_separation>0.32</wheel_separation>
+      <wheel_separation>0.34</wheel_separation>
       <wheel_radius>0.065</wheel_radius>
-      <max_wheel_torque>25.0</max_wheel_torque>
-      <max_linear_acceleration>2.5</max_linear_acceleration>
-      <max_angular_acceleration>3.5</max_angular_acceleration>
-      <min_linear_velocity>-1.0</min_linear_velocity>
-      <max_linear_velocity>1.0</max_linear_velocity>
-      <min_angular_velocity>-2.5</min_angular_velocity>
-      <max_angular_velocity>2.5</max_angular_velocity>
+      <max_wheel_torque>150.0</max_wheel_torque>
+      <max_linear_acceleration>5.0</max_linear_acceleration>
+      <max_angular_acceleration>8.0</max_angular_acceleration>
+      <min_linear_velocity>-1.5</min_linear_velocity>
+      <max_linear_velocity>1.5</max_linear_velocity>
+      <min_angular_velocity>-3.0</min_angular_velocity>
+      <max_angular_velocity>3.0</max_angular_velocity>
       <topic>/cmd_vel</topic>
       <odom_topic>/odom</odom_topic>

File: ros2_ws/src/gracemo_description/urdf/gracemo_vira.urdf.xacro (robot description, xacro)
@@ -96,12 +96,12 @@
       <origin xyz="0 ${y_offset} 0" rpy="0 0 0" />
       <axis xyz="0 1 0" />
-      <limit effort="50.0" velocity="20.0" />
-      <dynamics damping="0.02" friction="0.02" />
+      <limit effort="150.0" velocity="20.0" />
+      <dynamics damping="0.01" friction="0.01" />
     </joint>
     <gazebo reference="${prefix}_wheel_link">
-      <mu1>50.0</mu1>
-      <mu2>50.0</mu2>
+      <mu1>1.5</mu1>
+      <mu2>1.5</mu2>
       <kp>1000000.0</kp>
-      <kd>10.0</kd>
+      <kd>100.0</kd>
       <minDepth>0.001</minDepth>
       <material>Gazebo/DarkGrey</material>

Commit message: feat(manipulation): 7-DOF humanoid arm, slip-free DetachableJoint physics & staged verification ladder
- Add 7-DOF humanoid manipulator URDF with ball-and-socket shoulder, knuckle elbow, and compact gripper
- Implement 6D task-space DLS kinematic solver with nullspace torso repulsion & natural rest stances
- Integrate Gazebo Harmonic DetachableJoint plugin and high-friction contact surfaces for slip-free grasping
- Add comprehensive manipulation skill architecture: affordance synthesis, closed-loop verifier, and reflex shields
- Add third-person bedroom overview camera and staged verification ladder (G1 -> G2 -> G3 -> M4)
- Include MoveIt 2 TRAC-IK kinematics config, MNSE kernel ledger integration, and end-to-end test suite

File: ros2_ws/src/gracemo_description/urdf/gazebo_plugins.xacro (robot description, xacro)
@@ -5,4 +5,6 @@
   <!-- ======================================================================== -->
   <gazebo>
+    <!-- Contact Sensor System -->
+    <plugin filename="gz-sim-contact-system" name="gz::sim::systems::Contact" />
     <!-- Joint State Publisher -->
     <plugin filename="gz-sim-joint-state-publisher-system" name="gz::sim::systems::JointStatePublisher" />
@@ -80,4 +82,26 @@
   </gazebo>
   <!-- ======================================================================== -->
+  <!-- 3D Depth Camera Sensor Definition (Registered Volumetric Perception)     -->
+  <!-- ======================================================================== -->
+  <gazebo reference="camera_link">
+    <sensor name="depth_camera" type="depth_camera">
+      <pose>0 0 0 0 0 0</pose>
+      <topic>/camera/depth_image</topic>
+      <update_rate>15.0</update_rate>
+      <camera>
+        <horizontal_fov>1.15</horizontal_fov>
+        <image>
+          <width>320</width>
+          <height>240</height>
+        </image>
+        <clip>
+          <near>0.10</near>
+          <far>10.0</far>
+        </clip>
+      </camera>
+      <always_on>1</always_on>
+    </sensor>
+  </gazebo>
+  <!-- ======================================================================== -->
   <!-- IMU Sensor Definition                                                    -->
   <!-- ======================================================================== -->
@@ -89,3 +113,190 @@
     </sensor>
   </gazebo>
+  <!-- ======================================================================== -->
+  <!-- 360° Tactile Bumper Contact Sensor (Physical Collision Defense)           -->
+  <!-- ======================================================================== -->
+  <gazebo reference="bumper_link">
+    <sensor name="bumper_contact" type="contact">
+      <contact>
+        <collision>bumper_collision</collision>
+      </contact>
+      <topic>/bumper/contacts</topic>
+      <update_rate>50.0</update_rate>
+      <always_on>1</always_on>
+    </sensor>
+  </gazebo>
+  <!-- ======================================================================== -->
+  <!-- Corner ToF / Ultrasonic Proximity Sensors                                 -->
+  <!-- ======================================================================== -->
+  <xacro:macro name="tof_proximity_sensor" params="name reference topic">
+    <gazebo reference="${reference}">
+      <sensor name="${name}" type="gpu_lidar">
+        <pose>0 0 0 0 0 0</pose>
+        <topic>${topic}</topic>
+        <update_rate>25.0</update_rate>
+        <ray>
+          <scan>
+            <horizontal>
+              <samples>5</samples>
+              <resolution>1</resolution>
+              <min_angle>-0.15</min_angle>
+              <max_angle>0.15</max_angle>
+            </horizontal>
+          </scan>
+          <range>
+            <min>0.02</min>
+            <max>2.0</max>
+            <resolution>0.005</resolution>
+          </range>
+        </ray>
+        <always_on>1</always_on>
+      </sensor>
+    </gazebo>
+  </xacro:macro>
+  <xacro:tof_proximity_sensor name="tof_front_left" reference="tof_front_left_link" topic="/tof/front_left" />
+  <xacro:tof_proximity_sensor name="tof_front_right" reference="tof_front_right_link" topic="/tof/front_right" />
+  <xacro:tof_proximity_sensor name="tof_rear" reference="tof_rear_link" topic="/tof/rear" />
+  <!-- ======================================================================== -->
+  <!-- Hand Subsystem Plugins & Contacts                                        -->
+  <!-- ======================================================================== -->
+  <gazebo reference="finger_left_link">
+    <sensor name="hand_contact_left" type="contact">
+      <contact>
+        <collision>finger_left_collision</collision>
+      </contact>
+      <topic>/hand/contacts/left</topic>
+      <update_rate>50.0</update_rate>
+    </sensor>
+  </gazebo>
+  <gazebo reference="finger_right_link">
+    <sensor name="hand_contact_right" type="contact">
+      <contact>
+        <collision>finger_right_collision</collision>
+      </contact>
+      <topic>/hand/contacts/right</topic>
+      <update_rate>50.0</update_rate>
+    </sensor>
+  </gazebo>
+  <gazebo>
+    <!-- 6-DOF Right Arm Joint Position Controllers (Milestones M2 / M3) -->
+    <plugin
+      filename="gz-sim-joint-position-controller-system"
+      name="gz::sim::systems::JointPositionController">
+      <joint_name>right_shoulder_yaw_joint</joint_name>
+      <topic>/arm/joint_1/cmd_pos</topic>
+      <initial_position>0.0</initial_position>
+      <p_gain>800</p_gain>
+      <i_gain>10</i_gain>
+      <d_gain>30</d_gain>
+      <cmd_max>50</cmd_max>
+      <cmd_min>-50</cmd_min>
+    </plugin>
+    <plugin
+      filename="gz-sim-joint-position-controller-system"
+      name="gz::sim::systems::JointPositionController">
+      <joint_name>right_shoulder_pitch_joint</joint_name>
+      <topic>/arm/joint_2/cmd_pos</topic>
+      <initial_position>0.20</initial_position>
+      <p_gain>800</p_gain>
+      <i_gain>10</i_gain>
+      <d_gain>30</d_gain>
+      <cmd_max>50</cmd_max>
+      <cmd_min>-50</cmd_min>
+    </plugin>
+    <plugin
+      filename="gz-sim-joint-position-controller-system"
+      name="gz::sim::systems::JointPositionController">
+      <joint_name>right_shoulder_roll_joint</joint_name>
+      <topic>/arm/joint_3/cmd_pos</topic>
+      <initial_position>0.0</initial_position>
+      <p_gain>800</p_gain>
+      <i_gain>10</i_gain>
+      <d_gain>30</d_gain>
+      <cmd_max>50</cmd_max>
+      <cmd_min>-50</cmd_min>
+    </plugin>
+    <plugin
+      filename="gz-sim-joint-position-controller-system"
+      name="gz::sim::systems::JointPositionController">
+      <joint_name>right_elbow_pitch_joint</joint_name>
+      <topic>/arm/joint_4/cmd_pos</topic>
+      <initial_position>-1.80</initial_position>
+      <p_gain>600</p_gain>
+      <i_gain>8</i_gain>
+      <d_gain>20</d_gain>
+      <cmd_max>40</cmd_max>
+      <cmd_min>-40</cmd_min>
+    </plugin>
+    <plugin
+      filename="gz-sim-joint-position-controller-system"
+      name="gz::sim::systems::JointPositionController">
+      <joint_name>right_wrist_pitch_joint</joint_name>
+      <topic>/arm/joint_5/cmd_pos</topic>
+      <initial_position>0.60</initial_position>
+      <p_gain>400</p_gain>
+      <i_gain>5</i_gain>
+      <d_gain>10</d_gain>
+      <cmd_max>25</cmd_max>
+      <cmd_min>-25</cmd_min>
+    </plugin>
+    <plugin
+      filename="gz-sim-joint-position-controller-system"
+      name="gz::sim::systems::JointPositionController">
+      <joint_name>right_wrist_yaw_joint</joint_name>
+      <topic>/arm/joint_6/cmd_pos</topic>
+      <initial_position>0.0</initial_position>
+      <p_gain>400</p_gain>
+      <i_gain>5</i_gain>
+      <d_gain>10</d_gain>
+      <cmd_max>25</cmd_max>
+      <cmd_min>-25</cmd_min>
+    </plugin>
+    <plugin
+      filename="gz-sim-joint-position-controller-system"
+      name="gz::sim::systems::JointPositionController">
+      <joint_name>right_wrist_roll_joint</joint_name>
+      <topic>/arm/joint_7/cmd_pos</topic>
+      <initial_position>0.0</initial_position>
+      <p_gain>400</p_gain>
+      <i_gain>5</i_gain>
+      <d_gain>10</d_gain>
+      <cmd_max>25</cmd_max>
+      <cmd_min>-25</cmd_min>
+    </plugin>
+    <plugin
+      filename="gz-sim-joint-position-controller-system"
+      name="gz::sim::systems::JointPositionController">
+      <joint_name>finger_left_joint</joint_name>
+      <topic>/hand/left_finger/cmd_pos</topic>
+      <initial_position>0.001</initial_position>
+      <p_gain>2200</p_gain>
+      <i_gain>15</i_gain>
+      <d_gain>30</d_gain>
+      <cmd_max>120</cmd_max>
+      <cmd_min>-120</cmd_min>
+    </plugin>
+    <plugin
+      filename="gz-sim-joint-position-controller-system"
+      name="gz::sim::systems::JointPositionController">
+      <joint_name>finger_right_joint</joint_name>
+      <topic>/hand/right_finger/cmd_pos</topic>
+      <initial_position>0.001</initial_position>
+      <p_gain>2200</p_gain>
+      <i_gain>15</i_gain>
+      <d_gain>30</d_gain>
+      <cmd_max>120</cmd_max>
+      <cmd_min>-120</cmd_min>
+    </plugin>
+    <!-- Dynamic DetachableJoint Plugin for guaranteed slip-free picking -->
+    <plugin
+      filename="gz-sim-detachable-joint-system"
+      name="gz::sim::systems::DetachableJoint">
+      <parent_link>right_palm_link</parent_link>
+      <child_model>book_math</child_model>
+      <child_link>link</child_link>
+      <detach_topic>/gracemo_vira/detachable_joint/detach</detach_topic>
+      <attach_topic>/gracemo_vira/detachable_joint/attach</attach_topic>
+      <output_topic>/gracemo_vira/detachable_joint/state</output_topic>
+    </plugin>
+  </gazebo>
 </robot>
