Commit message: feat(manipulation): 7-DOF humanoid arm, slip-free DetachableJoint physics & staged verification ladder
- Add 7-DOF humanoid manipulator URDF with ball-and-socket shoulder, knuckle elbow, and compact gripper
- Implement 6D task-space DLS kinematic solver with nullspace torso repulsion & natural rest stances
- Integrate Gazebo Harmonic DetachableJoint plugin and high-friction contact surfaces for slip-free grasping
- Add comprehensive manipulation skill architecture: affordance synthesis, closed-loop verifier, and reflex shields
- Add third-person bedroom overview camera and staged verification ladder (G1 -> G2 -> G3 -> M4)
- Include MoveIt 2 TRAC-IK kinematics config, MNSE kernel ledger integration, and end-to-end test suite

File: ros2_ws/src/gracemo_description/urdf/gracemo_vira.urdf.xacro (robot description, xacro)
@@ -1,317 +1,741 @@
-<?xml version="1.0" ?>
-<!-- ============================================================================== -->
-<!-- GRaCEmo ViRa — Built on Industry-Standard TurtleBot3 Waffle Architecture       -->
-<!-- Factory-Calibrated Physics, Balanced Inertia, Zero-Friction Caster Dynamics   -->
-<!-- ============================================================================== -->
-<robot name="gracemo_vira" xmlns:xacro="http://ros.org/wiki/xacro">
-  <!-- Material Colors -->
-  <material name="black">
-    <color rgba="0.0 0.0 0.0 1.0"/>
-  </material>
-  <material name="dark">
-    <color rgba="0.2 0.2 0.2 1.0"/>
-  </material>
-  <material name="light_black">
-    <color rgba="0.3 0.3 0.3 1.0"/>
-  </material>
-  <material name="chassis_blue">
-    <color rgba="0.0 0.6 0.9 1.0"/>
-  </material>
-  <material name="white">
-    <color rgba="1.0 1.0 1.0 1.0"/>
-  </material>
+<?xml version="1.0"?>
+<robot name="gracemo_vira" xmlns:xacro="http://www.ros.org/wiki/xacro">
+  <!-- Include sub-files -->
+  <xacro:include filename="$(find gracemo_description)/urdf/materials.xacro" />
+  <xacro:include filename="$(find gracemo_description)/urdf/gazebo_plugins.xacro" />
+  <!-- Dimensions & Constants -->
+  <xacro:property name="wheel_radius" value="0.065" />
+  <xacro:property name="wheel_width" value="0.030" />
+  <xacro:property name="wheelbase" value="0.34" />
+  <xacro:property name="chassis_radius" value="0.19" />
+  <xacro:property name="chassis_height" value="0.14" />
+  <xacro:property name="torso_height" value="0.40" />
+  <xacro:property name="torso_width" value="0.20" />
+  <xacro:property name="torso_depth" value="0.16" />
   <!-- Base Footprint (Ground Projection) -->
-  <link name="base_footprint"/>
-  <joint name="base_joint" type="fixed">
-    <parent link="base_footprint"/>
+  <link name="base_footprint" />
+  <joint name="base_footprint_joint" type="fixed">
+    <parent link="base_footprint" />
     <child link="base_link" />
-    <origin xyz="0 0 0.010" rpy="0 0 0"/>
-  </joint>
-  <!-- Base Link (Chassis) -->
+    <origin xyz="0 0 ${wheel_radius}" rpy="0 0 0" />
+  </joint>
+  <!-- ======================================================================== -->
+  <!-- Base Link (Sleek Mobile Chassis with Non-Overlapping Collision)          -->
+  <!-- ======================================================================== -->
   <link name="base_link">
-    <visual>
-      <origin xyz="-0.064 0 0.0" rpy="0 0 0"/>
-      <geometry>
-        <mesh filename="package://turtlebot3_description/meshes/bases/waffle_base.stl" scale="0.001 0.001 0.001"/>
-      </geometry>
-      <material name="chassis_blue"/>
+    <!-- Visual Shell -->
+    <visual>
+      <origin xyz="0 0 ${chassis_height/2.0}" rpy="0 0 0" />
+      <geometry>
+        <cylinder radius="${chassis_radius}" length="${chassis_height}" />
+      </geometry>
+      <material name="chassis_blue" />
+    </visual>
+    <!-- Lower Protective Skirt -->
+    <visual>
+      <origin xyz="0 0 ${chassis_height * 0.2}" rpy="0 0 0" />
+      <geometry>
+        <cylinder radius="${chassis_radius + 0.005}" length="${chassis_height * 0.35}" />
+      </geometry>
+      <material name="dark_grey" />
+    </visual>
+    <!-- Top Deck Plate -->
+    <visual>
+      <origin xyz="0 0 ${chassis_height + 0.005}" rpy="0 0 0" />
+      <geometry>
+        <cylinder radius="${chassis_radius * 0.9}" length="0.01" />
+      </geometry>
+      <material name="dark_grey" />
     </visual>
     <collision>
-      <origin xyz="-0.064 0 0.047" rpy="0 0 0"/>
-      <geometry>
-        <box size="0.266 0.266 0.094"/>
+      <origin xyz="0 0 ${chassis_height/2.0 + 0.01}" rpy="0 0 0" />
+      <geometry>
+        <box size="0.24 0.20 ${chassis_height}" />
       </geometry>
     </collision>
-    <inertial>
-      <origin xyz="0 0 0" rpy="0 0 0"/>
-      <mass value="1.3729096"/>
-      <inertia ixx="8.7002718e-03" ixy="-4.7576583e-05" ixz="1.1160499e-04"
-               iyy="8.6195418e-03" iyz="-3.5422299e-06"
-               izz="1.4612727e-02" />
-    </inertial>
-  </link>
-  <!-- Left Drive Wheel -->
-  <joint name="wheel_left_joint" type="continuous">
-    <parent link="base_link"/>
-    <child link="wheel_left_link"/>
-    <origin xyz="0.0 0.144 0.023" rpy="-1.57 0 0"/>
-    <axis xyz="0 0 1"/>
-  </joint>
-  <link name="wheel_left_link">
-    <visual>
-      <origin xyz="0 0 0" rpy="1.57 0 0"/>
-      <geometry>
-        <mesh filename="package://turtlebot3_description/meshes/wheels/left_tire.stl" scale="0.001 0.001 0.001"/>
-      </geometry>
-      <material name="dark"/>
+    <!-- Heavy low base mass to keep wheels firmly planted with high traction -->
+    <inertial>
+      <origin xyz="0 0 0.02" rpy="0 0 0" />
+      <mass value="8.0" />
+      <inertia ixx="0.04" ixy="0.0" ixz="0.0" iyy="0.04" iyz="0.0" izz="0.06" />
+    </inertial>
+  </link>
+  <!-- ======================================================================== -->
+  <!-- 360° Tactile Bumper Ring (Physical Contact Sensor & RGB Halo)            -->
+  <!-- ======================================================================== -->
+  <link name="bumper_link">
+    <visual>
+      <origin xyz="0 0 0" rpy="0 0 0" />
+      <geometry>
+        <cylinder radius="0.205" length="0.04" />
+      </geometry>
+      <material name="cyan_glow" />
+    </visual>
+    <collision name="bumper_collision">
+      <origin xyz="0 0 0" rpy="0 0 0" />
+      <geometry>
+        <cylinder radius="0.205" length="0.04" />
+      </geometry>
+    </collision>
+    <inertial>
+      <mass value="0.2" />
+      <inertia ixx="0.001" ixy="0.0" ixz="0.0" iyy="0.001" iyz="0.0" izz="0.001" />
+    </inertial>
+  </link>
+  <joint name="bumper_joint" type="fixed">
+    <parent link="base_link" />
+    <child link="bumper_link" />
+    <origin xyz="0 0 0.04" rpy="0 0 0" />
+  </joint>
+  <!-- ======================================================================== -->
+  <!-- Corner ToF / Ultrasonic Proximity Sensor Mounts                          -->
+  <!-- ======================================================================== -->
+  <link name="tof_front_left_link">
+    <inertial><mass value="0.01"/><inertia ixx="0.00001" ixy="0" ixz="0" iyy="0.00001" iyz="0" izz="0.00001"/></inertial>
+  </link>
+  <joint name="tof_front_left_joint" type="fixed">
+    <parent link="base_link" />
+    <child link="tof_front_left_link" />
+    <origin xyz="0.16 0.12 0.08" rpy="0 0 0.7854" />
+  </joint>
+  <link name="tof_front_right_link">
+    <inertial><mass value="0.01"/><inertia ixx="0.00001" ixy="0" ixz="0" iyy="0.00001" iyz="0" izz="0.00001"/></inertial>
+  </link>
+  <joint name="tof_front_right_joint" type="fixed">
+    <parent link="base_link" />
+    <child link="tof_front_right_link" />
+    <origin xyz="0.16 -0.12 0.08" rpy="0 0 -0.7854" />
+  </joint>
+  <link name="tof_rear_link">
+    <inertial><mass value="0.01"/><inertia ixx="0.00001" ixy="0" ixz="0" iyy="0.00001" iyz="0" izz="0.00001"/></inertial>
+  </link>
+  <joint name="tof_rear_joint" type="fixed">
+    <parent link="base_link" />
+    <child link="tof_rear_link" />
+    <origin xyz="-0.18 0 0.08" rpy="0 0 3.14159" />
+  </joint>
+  <!-- ======================================================================== -->
+  <!-- Drive Wheels (High Grip & Smooth Rolling)                                -->
+  <!-- ======================================================================== -->
+  <xacro:macro name="wheel" params="prefix y_offset">
+    <link name="${prefix}_wheel_link">
+      <visual>
+        <origin xyz="0 0 0" rpy="${pi/2} 0 0" />
+        <geometry>
+          <cylinder radius="${wheel_radius}" length="${wheel_width}" />
+        </geometry>
+        <material name="rubber_black" />
+      </visual>
+      <visual>
+        <origin xyz="0 0 0" rpy="${pi/2} 0 0" />
+        <geometry>
+          <cylinder radius="${wheel_radius * 0.6}" length="${wheel_width + 0.002}" />
+        </geometry>
+        <material name="metallic_silver" />
+      </visual>
+      <collision>
+        <origin xyz="0 0 0" rpy="${pi/2} 0 0" />
+        <geometry>
+          <cylinder radius="${wheel_radius}" length="${wheel_width}" />
+        </geometry>
+      </collision>
+      <inertial>
+        <mass value="0.8" />
+        <inertia ixx="0.001" ixy="0.0" ixz="0.0" iyy="0.001" iyz="0.0" izz="0.001" />
+      </inertial>
+    </link>
+    <joint name="${prefix}_wheel_joint" type="continuous">
+      <parent link="base_link" />
+      <child link="${prefix}_wheel_link" />
+      <origin xyz="0 ${y_offset} 0" rpy="0 0 0" />
+      <axis xyz="0 1 0" />
+      <limit effort="150.0" velocity="20.0" />
+      <dynamics damping="1.5" friction="1.5" />
+    </joint>
+    <gazebo reference="${prefix}_wheel_link">
+      <mu1>1.5</mu1>
+      <mu2>1.5</mu2>
+      <kp>1000000.0</kp>
+      <kd>100.0</kd>
+      <minDepth>0.001</minDepth>
+      <material>Gazebo/DarkGrey</material>
+    </gazebo>
+  </xacro:macro>
+  <xacro:wheel prefix="left" y_offset="${wheelbase/2.0}" />
+  <xacro:wheel prefix="right" y_offset="${-wheelbase/2.0}" />
+  <!-- ======================================================================== -->
+  <!-- Support Casters (Exact ground tangent frictionless gliders)              -->
+  <!-- ======================================================================== -->
+  <xacro:macro name="caster" params="prefix x_offset">
+    <link name="${prefix}_caster_link">
+      <visual>
+        <geometry>
+          <sphere radius="0.025" />
+        </geometry>
+        <material name="metallic_silver" />
+      </visual>
+      <collision>
+        <geometry>
+          <sphere radius="0.025" />
+        </geometry>
+      </collision>
+      <inertial>
+        <mass value="0.05" />
+        <inertia ixx="0.00001" ixy="0.0" ixz="0.0" iyy="0.00001" iyz="0.0" izz="0.00001" />
+      </inertial>
+    </link>
+    <joint name="${prefix}_caster_joint" type="fixed">
+      <parent link="base_link" />
+      <child link="${prefix}_caster_link" />
+      <origin xyz="${x_offset} 0 ${-wheel_radius + 0.025}" rpy="0 0 0" />
+    </joint>
+    <gazebo reference="${prefix}_caster_link">
+      <mu1>0.0</mu1>
+      <mu2>0.0</mu2>
+      <kp>1000000.0</kp>
+      <kd>10.0</kd>
+      <minDepth>0.0001</minDepth>
+      <material>Gazebo/Grey</material>
+    </gazebo>
+  </xacro:macro>
+  <xacro:caster prefix="front" x_offset="0.14" />
+  <xacro:caster prefix="rear" x_offset="-0.14" />
+  <!-- ======================================================================== -->
+  <!-- Humanoid Torso (Visual Only — Collision handled by unified base)         -->
+  <!-- ======================================================================== -->
+  <link name="torso_link">
+    <visual>
+      <origin xyz="0 0 ${torso_height/2.0}" rpy="0 0 0" />
+      <geometry>
+        <box size="${torso_depth} ${torso_width} ${torso_height}" />
+      </geometry>
+      <material name="chassis_blue" />
+    </visual>
+    <visual>
+      <origin xyz="${torso_depth/2.0 + 0.004} 0 ${torso_height * 0.6}" rpy="0 0 0" />
+      <geometry>
+        <box size="0.006 0.13 0.11" />
+      </geometry>
+      <material name="camera_lens_black" />
+    </visual>
+    <inertial>
+      <origin xyz="0 0 0.05" rpy="0 0 0" />
+      <mass value="0.3" />
+      <inertia ixx="0.001" ixy="0.0" ixz="0.0" iyy="0.001" iyz="0.0" izz="0.001" />
+    </inertial>
+  </link>
+  <joint name="torso_joint" type="fixed">
+    <parent link="base_link" />
+    <child link="torso_link" />
+    <origin xyz="-0.02 0 ${chassis_height}" rpy="0 0 0" />
+  </joint>
+  <!-- ======================================================================== -->
+  <!-- 2D LiDAR Sensor                                                          -->
+  <!-- ======================================================================== -->
+  <link name="lidar_link">
+    <visual>
+      <origin xyz="0 0 0.015" rpy="0 0 0" />
+      <geometry>
+        <cylinder radius="0.045" length="0.03" />
+      </geometry>
+      <material name="dark_grey" />
+    </visual>
+    <visual>
+      <origin xyz="0 0 0.032" rpy="0 0 0" />
+      <geometry>
+        <cylinder radius="0.04" length="0.015" />
+      </geometry>
+      <material name="lidar_orange" />
+    </visual>
+    <inertial>
+      <origin xyz="0 0 0.02" rpy="0 0 0" />
+      <mass value="0.2" />
+      <inertia ixx="0.0001" ixy="0.0" ixz="0.0" iyy="0.0001" iyz="0.0" izz="0.0001" />
+    </inertial>
+  </link>
+  <joint name="lidar_joint" type="fixed">
+    <parent link="base_link" />
+    <child link="lidar_link" />
+    <origin xyz="0.11 0 ${chassis_height}" rpy="0 0 0" />
+  </joint>
+  <!-- ======================================================================== -->
+  <!-- Humanoid Head & Camera                                                   -->
+  <!-- ======================================================================== -->
+  <link name="head_link">
+    <visual>
+      <origin xyz="0 0 0.02" rpy="0 0 0" />
+      <geometry>
+        <cylinder radius="0.035" length="0.04" />
+      </geometry>
+      <material name="dark_grey" />
+    </visual>
+    <visual>
+      <origin xyz="0.01 0 0.09" rpy="0 0 0" />
+      <geometry>
+        <box size="0.14 0.16 0.11" />
+      </geometry>
+      <material name="chassis_blue" />
+    </visual>
+    <visual>
+      <origin xyz="0.081 0 0.09" rpy="0 0 0" />
+      <geometry>
+        <box size="0.006 0.13 0.07" />
+      </geometry>
+      <material name="camera_lens_black" />
+    </visual>
+    <inertial>
+      <origin xyz="0.01 0 0.08" rpy="0 0 0" />
+      <mass value="0.5" />
+      <inertia ixx="0.001" ixy="0.0" ixz="0.0" iyy="0.001" iyz="0.0" izz="0.001" />
+    </inertial>
+  </link>
+  <joint name="head_joint" type="fixed">
+    <parent link="torso_link" />
+    <child link="head_link" />
+    <origin xyz="0 0 ${torso_height}" rpy="0 0 0" />
+  </joint>
+  <link name="camera_link">
+    <visual>
+      <origin xyz="0 0 0" rpy="0 ${pi/2} 0" />
+      <geometry>
+        <cylinder radius="0.012" length="0.01" />
+      </geometry>
+      <material name="metallic_silver" />
+    </visual>
+  </link>
+  <joint name="camera_joint" type="fixed">
+    <parent link="head_link" />
+    <child link="camera_link" />
+    <origin xyz="0.085 0 0.09" rpy="0 0 0" />
+  </joint>
+  <link name="camera_optical_link" />
+  <joint name="camera_optical_joint" type="fixed">
+    <parent link="camera_link" />
+    <child link="camera_optical_link" />
+    <origin xyz="0 0 0" rpy="${-pi/2} 0 ${-pi/2}" />
+  </joint>
+  <!-- ======================================================================== -->
+  <!-- Manipulation Arm Pods (Visual Only)                                      -->
+  <!-- ======================================================================== -->
+  <!-- Left Arm Pod (Visual Only) -->
+  <link name="left_arm_link">
+    <visual>
+      <origin xyz="0 0 -0.09" rpy="0 0 0" />
+      <geometry>
+        <box size="0.045 0.035 0.18" />
+      </geometry>
+      <material name="metallic_silver" />
+    </visual>
+    <inertial>
+      <origin xyz="0 0 -0.09" rpy="0 0 0" />
+      <mass value="0.2" />
+      <inertia ixx="0.001" ixy="0.0" ixz="0.0" iyy="0.001" iyz="0.0" izz="0.001" />
+    </inertial>
+  </link>
+  <joint name="left_arm_joint" type="fixed">
+    <parent link="torso_link" />
+    <child link="left_arm_link" />
+    <origin xyz="0.0 ${torso_width/2.0 + 0.022} ${torso_height - 0.04}" rpy="0 0 0" />
+  </joint>
+  <!-- ======================================================================== -->
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
File: ros2_ws/src/gracemo_description/urdf/materials.xacro (robot description, xacro)
@@ -19,3 +19,12 @@
     <color rgba="0.95 0.45 0.05 1.0"/>
   </material>
+  <material name="cyan_glow">
+    <color rgba="0.0 0.83 1.0 1.0"/>
+  </material>
+  <material name="matte_dark_titanium">
+    <color rgba="0.12 0.14 0.17 1.0"/>
+  </material>
+  <material name="safety_orange">
+    <color rgba="1.0 0.40 0.0 1.0"/>
+  </material>
 </robot>

Commit message: fix(nav+arm): posture arm in natural mid-torso tuck, orient into room on arrival, and add caster mounts

File: ros2_ws/src/gracemo_description/urdf/gazebo_plugins.xacro (robot description, xacro)
@@ -197,4 +197,16 @@
       <joint_name>right_shoulder_pitch_joint</joint_name>
       <topic>/arm/joint_2/cmd_pos</topic>
+      <initial_position>0.90</initial_position>
+      <p_gain>800</p_gain>
+      <i_gain>10</i_gain>
+      <d_gain>30</d_gain>
+      <cmd_max>50</cmd_max>
+      <cmd_min>-50</cmd_min>
+    </plugin>
+    <plugin
+      filename="gz-sim-joint-position-controller-system"
+      name="gz::sim::systems::JointPositionController">
+      <joint_name>right_shoulder_roll_joint</joint_name>
+      <topic>/arm/joint_3/cmd_pos</topic>
       <initial_position>0.20</initial_position>
       <p_gain>800</p_gain>
@@ -207,19 +219,7 @@
       filename="gz-sim-joint-position-controller-system"
       name="gz::sim::systems::JointPositionController">
-      <joint_name>right_shoulder_roll_joint</joint_name>
-      <topic>/arm/joint_3/cmd_pos</topic>
-      <initial_position>0.0</initial_position>
-      <p_gain>800</p_gain>
-      <i_gain>10</i_gain>
-      <d_gain>30</d_gain>
-      <cmd_max>50</cmd_max>
-      <cmd_min>-50</cmd_min>
-    </plugin>
-    <plugin
-      filename="gz-sim-joint-position-controller-system"
-      name="gz::sim::systems::JointPositionController">
       <joint_name>right_elbow_pitch_joint</joint_name>
       <topic>/arm/joint_4/cmd_pos</topic>
-      <initial_position>-1.80</initial_position>
+      <initial_position>-1.25</initial_position>
       <p_gain>600</p_gain>
       <i_gain>8</i_gain>

File: ros2_ws/src/gracemo_description/urdf/gracemo_vira.urdf.xacro (robot description, xacro)
@@ -169,9 +169,19 @@
   <xacro:macro name="caster" params="prefix x_offset">
     <link name="${prefix}_caster_link">
+      <!-- Rolling Caster Ball -->
       <visual>
+        <origin xyz="0 0 0" rpy="0 0 0" />
         <geometry>
           <sphere radius="0.025" />
         </geometry>
         <material name="metallic_silver" />
+      </visual>
+      <!-- Caster Mounting Housing / Bracket (solidly connects ball to chassis underside) -->
+      <visual>
+        <origin xyz="0 0 0.022" rpy="0 0 0" />
+        <geometry>
+          <cylinder radius="0.022" length="0.035" />
+        </geometry>
+        <material name="dark_grey" />
       </visual>
       <collision>
