Commit message: feat: complete gracemo vira system with interaction engine, ros2 bridge, and perception controllers

File: ros2_ws/src/gracemo_description/urdf/gazebo_plugins.xacro (robot description, xacro)
@@ -179,4 +179,29 @@
   </gazebo>
   <gazebo>
+    <!-- 2-DOF Active Head / Neck Joint Position Controllers -->
+    <plugin
+      filename="gz-sim-joint-position-controller-system"
+      name="gz::sim::systems::JointPositionController">
+      <joint_name>neck_pan_joint</joint_name>
+      <topic>/head/pan/cmd_pos</topic>
+      <initial_position>0.0</initial_position>
+      <p_gain>180</p_gain>
+      <i_gain>2</i_gain>
+      <d_gain>12</d_gain>
+      <cmd_max>20</cmd_max>
+      <cmd_min>-20</cmd_min>
+    </plugin>
+    <plugin
+      filename="gz-sim-joint-position-controller-system"
+      name="gz::sim::systems::JointPositionController">
+      <joint_name>neck_tilt_joint</joint_name>
+      <topic>/head/tilt/cmd_pos</topic>
+      <initial_position>0.0</initial_position>
+      <p_gain>180</p_gain>
+      <i_gain>2</i_gain>
+      <d_gain>12</d_gain>
+      <cmd_max>20</cmd_max>
+      <cmd_min>-20</cmd_min>
+    </plugin>
     <!-- 6-DOF Right Arm Joint Position Controllers (Milestones M2 / M3) -->
     <plugin

File: ros2_ws/src/gracemo_description/urdf/gracemo_vira.urdf.xacro (robot description, xacro)
@@ -48,8 +48,8 @@
       <material name="dark_grey" />
     </visual>
-    <collision>
-      <origin xyz="0 0 ${chassis_height/2.0 + 0.01}" rpy="0 0 0" />
-      <geometry>
-        <box size="0.24 0.20 ${chassis_height}" />
+    <collision name="base_link_collision">
+      <origin xyz="0 0 0.08" rpy="0 0 0" />
+      <geometry>
+        <cylinder radius="${chassis_radius}" length="0.12" />
       </geometry>
     </collision>
@@ -229,4 +229,10 @@
       <material name="camera_lens_black" />
     </visual>
+    <collision name="torso_collision">
+      <origin xyz="0 0 ${torso_height/2.0}" rpy="0 0 0" />
+      <geometry>
+        <box size="${torso_depth} ${torso_width} ${torso_height}" />
+      </geometry>
+    </collision>
     <inertial>
       <origin xyz="0 0 0.05" rpy="0 0 0" />
@@ -258,4 +264,10 @@
       <material name="lidar_orange" />
     </visual>
+    <collision name="lidar_collision">
+      <origin xyz="0 0 0.015" rpy="0 0 0" />
+      <geometry>
+        <cylinder radius="0.045" length="0.03" />
+      </geometry>
+    </collision>
     <inertial>
       <origin xyz="0 0 0.02" rpy="0 0 0" />
@@ -270,16 +282,50 @@
   </joint>
   <!-- ======================================================================== -->
-  <!-- Humanoid Head & Camera                                                   -->
-  <!-- ======================================================================== -->
+  <!-- 2-DOF Active Articulated Head & Neck Assembly                            -->
+  <!-- ======================================================================== -->
+  <!-- Joint 1: Neck Pan Joint (Yaw around vertical Z-axis, ±120°) -->
+  <joint name="neck_pan_joint" type="revolute">
+    <parent link="torso_link" />
+    <child link="neck_pan_link" />
+    <origin xyz="0 0 ${torso_height}" rpy="0 0 0" />
+    <axis xyz="0 0 1" />
+    <limit lower="-2.0944" upper="2.0944" effort="25.0" velocity="3.0" />
+    <dynamics damping="0.2" friction="0.05" />
+  </joint>
+  <!-- Intermediate Neck Pan Turntable Collar Link -->
+  <link name="neck_pan_link">
+    <visual>
+      <origin xyz="0 0 0.02" rpy="0 0 0" />
+      <geometry>
+        <cylinder radius="0.035" length="0.04" />
+      </geometry>
+      <material name="dark_grey" />
+    </visual>
+    <collision name="neck_pan_collision">
+      <origin xyz="0 0 0.02" rpy="0 0 0" />
+      <geometry>
+        <cylinder radius="0.035" length="0.04" />
+      </geometry>
+    </collision>
+    <inertial>
+      <origin xyz="0 0 0.02" rpy="0 0 0" />
+      <mass value="0.15" />
+      <inertia ixx="0.0001" ixy="0.0" ixz="0.0" iyy="0.0001" iyz="0.0" izz="0.0001" />
+    </inertial>
+  </link>
+  <!-- Joint 2: Neck Tilt Joint (Pitch around lateral Y-axis, ±45°) -->
+  <joint name="neck_tilt_joint" type="revolute">
+    <parent link="neck_pan_link" />
+    <child link="head_link" />
+    <origin xyz="0 0 0.04" rpy="0 0 0" />
+    <axis xyz="0 1 0" />
+    <limit lower="-0.7854" upper="0.7854" effort="25.0" velocity="3.0" />
+    <dynamics damping="0.2" friction="0.05" />
+  </joint>
+  <!-- Articulated Humanoid Head Body Link -->
   <link name="head_link">
-    <visual>
-      <origin xyz="0 0 0.02" rpy="0 0 0" />
-      <geometry>
-        <cylinder radius="0.035" length="0.04" />
-      </geometry>
-      <material name="dark_grey" />
-    </visual>
-    <visual>
-      <origin xyz="0.01 0 0.09" rpy="0 0 0" />
+    <!-- Head Visual Shell -->
+    <visual>
+      <origin xyz="0.01 0 0.05" rpy="0 0 0" />
       <geometry>
         <box size="0.14 0.16 0.11" />
@@ -287,6 +333,7 @@
       <material name="chassis_blue" />
     </visual>
-    <visual>
-      <origin xyz="0.081 0 0.09" rpy="0 0 0" />
+    <!-- Front Sensor Visor Display Face -->
+    <visual>
+      <origin xyz="0.081 0 0.05" rpy="0 0 0" />
       <geometry>
         <box size="0.006 0.13 0.07" />
@@ -294,15 +341,17 @@
       <material name="camera_lens_black" />
     </visual>
-    <inertial>
-      <origin xyz="0.01 0 0.08" rpy="0 0 0" />
-      <mass value="0.5" />
+    <!-- Preserved Head Collision Geometry -->
+    <collision name="head_collision">
+      <origin xyz="0.01 0 0.05" rpy="0 0 0" />
+      <geometry>
+        <box size="0.14 0.16 0.11" />
+      </geometry>
+    </collision>
+    <inertial>
+      <origin xyz="0.01 0 0.04" rpy="0 0 0" />
+      <mass value="0.40" />
       <inertia ixx="0.001" ixy="0.0" ixz="0.0" iyy="0.001" iyz="0.0" izz="0.001" />
     </inertial>
   </link>
-  <joint name="head_joint" type="fixed">
-    <parent link="torso_link" />
-    <child link="head_link" />
-    <origin xyz="0 0 ${torso_height}" rpy="0 0 0" />
-  </joint>
   <link name="camera_link">
     <visual>
@@ -313,9 +362,15 @@
       <material name="metallic_silver" />
     </visual>
+    <collision name="camera_collision">
+      <origin xyz="0 0 0" rpy="0 ${pi/2} 0" />
+      <geometry>
+        <cylinder radius="0.012" length="0.01" />
+      </geometry>
+    </collision>
   </link>
   <joint name="camera_joint" type="fixed">
     <parent link="head_link" />
     <child link="camera_link" />
-    <origin xyz="0.085 0 0.09" rpy="0 0 0" />
+    <origin xyz="0.085 0 0.05" rpy="0 0 0" />
   </joint>
   <link name="camera_optical_link" />
@@ -337,4 +392,10 @@
       <material name="metallic_silver" />
     </visual>
+    <collision name="left_arm_collision">
+      <origin xyz="0 0 -0.09" rpy="0 0 0" />
+      <geometry>
+        <box size="0.045 0.035 0.18" />
+      </geometry>
+    </collision>
     <inertial>
       <origin xyz="0 0 -0.09" rpy="0 0 0" />
@@ -369,4 +430,10 @@
       <material name="dark_grey" />
     </visual>
+    <collision name="right_shoulder_yaw_collision">
+      <origin xyz="0 0 0" rpy="0 0 0" />
+      <geometry>
+        <sphere radius="0.038" />
+      </geometry>
+    </collision>
     <inertial>
       <mass value="0.15" />
@@ -400,4 +467,10 @@
       <material name="matte_dark_titanium" />
     </visual>
+    <collision name="right_shoulder_pitch_collision">
+      <origin xyz="0 0 0" rpy="0 0 0" />
+      <geometry>
+        <sphere radius="0.034" />
+      </geometry>
+    </collision>
     <inertial>
       <mass value="0.15" />
@@ -528,4 +601,10 @@
       <material name="metallic_silver" />
     </visual>
+    <collision name="right_wrist_pitch_collision">
+      <origin xyz="0 0 0" rpy="0 ${pi/2} 0" />
+      <geometry>
+        <cylinder radius="0.020" length="0.025" />
+      </geometry>
+    </collision>
     <inertial>
       <origin xyz="0 0 0" rpy="0 0 0" />
@@ -551,4 +630,10 @@
       <material name="matte_dark_titanium" />
     </visual>
+    <collision name="right_wrist_yaw_collision">
+      <origin xyz="0 0 0" rpy="0 0 0" />
+      <geometry>
+        <cylinder radius="0.018" length="0.020" />
+      </geometry>
+    </collision>
     <inertial>
       <origin xyz="0 0 0" rpy="0 0 0" />
