Commit message: feat(baseline): preserve accepted autonomous navigation and simulation substrate baseline
- Multi-room autonomous navigation verified across all six canonical apartment destinations
- 11-stage autonomous system readiness & lifecycle verified with 0 orphan processes
- Blender-derived 3D meshes, URDF, and Gazebo Harmonic apartment simulation integrated
- Single-owner velocity pipeline and real-time safety e-stop arbitration verified
- Hardware safety locks preserved: SerialMCUTransport.PROTOCOL_CONFIRMED=False, MOTOR_OUTPUT_ENABLED=0
- Full automated test suite passes (433 passed, 1 skipped)
- Baseline accepted prior to GUI development initiation

File: ros2_ws/src/gracemo_description/urdf/materials.xacro (robot description, xacro)
@@ -26,5 +26,11 @@
   </material>
   <material name="safety_orange">
-    <color rgba="1.0 0.40 0.0 1.0"/>
+    <color rgba="1.0 0.4745 0.0 1.0"/>
+  </material>
+  <material name="accent_orange">
+    <color rgba="1.0 0.4745 0.0 1.0"/>
+  </material>
+  <material name="pure_white">
+    <color rgba="0.96 0.96 0.96 1.0"/>
   </material>
 </robot>
